File: board/tex.brd (EAGLE design)
At the start: 150 x 100 mm, 179 parts, among them U2 RTC-DS1337S, Y1 32.768KHz

Commit message: continuing work on sch
Parts:
- removed JBATT, JGND, JP5, JP6, JP7, JP8: (no value), holla:1X05-1.27MM
- added D24, D25, D26, D27, D32, D33, D34, D35: (no value), holla:LED0603
- added D28, D29, D30, D31: (no value), holla:SOD-523
- added J1: (no value), holla:CONN-OSTT702
- added J11, J12, J13, J14: (no value), holla:1984620
- added J2, J3, J4, J5, J6, J7, J8, J9: (no value), holla:1984633
- added JP9: DNP, holla:PAD-JUMPER-2-NO_NO_SILK
- added K1, K2, K3, K4: HLS8L-DC5V-S-C, holla:REY5-19.0X15.0X15.0MM
- added Q37, Q38, Q39, Q40, Q41, Q42, Q43, Q44, Q45, Q46: (no value), holla:SOT23-3
- added R66: 1k, holla:R0603
- added R67, R68: 3.9k, holla:R0603
- added R69, R70, R71, R72, R73, R74, R75, R76, R77, R78, R80, R81, R82, R83, R84, R85, R86, R87: (no value), holla:R0603
- added R79: (no value), holla:R1210
- added U14: 24LC32A, holla:SO08
- added U15, U16, U17, U18: OPTO-LTV817, holla:LTV817
- moved R33 1309.6 mm to (571.5, 149.9)
- moved C17 1307.6 mm to (563.9, 138.4)
- moved R57 1305.5 mm to (652.0, 109.5), turned to 270 degrees
- moved R32 1303.3 mm to (558.8, 142.2)
- moved D19 1301.4 mm to (653.0, 106.5), turned to 90 degrees
- moved R55 1296.8 mm to (648.5, 109.5), turned to 270 degrees
- moved R64 1293.4 mm to (681.0, 113.0)
- moved D18 1292.7 mm to (649.5, 106.5), turned to 90 degrees
- moved R31 1288.7 mm to (558.8, 146.1)
- moved D22 1287.6 mm to (677.5, 112.0), turned to 90 degrees
- moved D23 1285.8 mm to (677.5, 113.5), turned to 270 degrees
- moved D21 1278.2 mm to (670.5, 112.0), turned to 90 degrees
- moved D20 1275.4 mm to (670.5, 113.5), turned to 270 degrees
- moved C15 1274.0 mm to (522.0, 139.7)
- moved R30 1273.0 mm to (528.3, 157.5)
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Connections:
- removed net N$76: D16.A, R51.1
- new net DCMOTOR1ENCA: U15.4
- new net DCMOTOR1ENCB: U16.4
- new net DCMOTOR2ENCA: U17.4
- new net DCMOTOR2ENCB: U18.4
- new net GND4: D31.A, D35.C, K4.3, Q46.3
- new net ID_SC: PCB1.P$28, R67.1, U14.6
- new net ID_SD: PCB1.P$27, R68.1, U14.5
- new net N$102: PCB1.P$2
- new net N$103: PCB1.P$4
- new net N$104: JP9.2, R66.1, U14.7
- new net N$106: PCB1.P$6
- new net N$108: PCB1.P$8
- new net N$109: PCB1.P$10
- new net N$110: PCB1.P$12
- new net N$111: PCB1.P$14
- new net N$112: PCB1.P$16
- new net N$113: PCB1.P$18
- new net N$114: PCB1.P$20
- new net N$115: PCB1.P$22
- new net N$116: PCB1.P$24
- new net N$117: PCB1.P$26
- new net N$118: PCB1.P$30
- new net N$119: PCB1.P$32
- new net N$120: PCB1.P$34
- new net N$121: PCB1.P$36
- new net N$122: PCB1.P$38
- new net N$123: PCB1.P$40
- new net N$124: PCB1.P$39
- new net N$125: PCB1.P$37
- new net N$126: PCB1.P$35
- new net N$127: PCB1.P$33
- new net N$128: PCB1.P$31
- new net N$129: PCB1.P$29
- new net N$130: PCB1.P$25
- new net N$131: PCB1.P$23
- new net N$132: PCB1.P$21
- new net N$133: PCB1.P$19
- new net N$134: PCB1.P$17
- new net N$135: PCB1.P$15
- new net N$136: PCB1.P$13
- new net N$137: PCB1.P$11
- new net N$138: PCB1.P$9
- new net N$139: D17.C, R53.2
- new net N$140: D16.C, R51.2
- new net N$141: D15.C, R49.2
- new net N$142: D14.C, R47.2
- new net N$143: J14.2, K1.1
- new net N$144: J14.1, K1.4
- new net N$145: J14.3, K1.5
- new net N$146: D13.C, R45.2
- new net N$147: D33.A, R85.1
- new net N$148: R80.1, U15.1
- new net N$149: J8.3, R81.2
- new net N$150: J8.2, R80.2
- new net N$151: J6.4, Q39.3
- new net N$152: J7.2, Q40.3
- new net N$153: J7.3, Q41.3
- new net N$154: J7.4, Q42.3
- new net N$155: R81.1, U16.1
- new net N$156: J9.2, R82.2
- new net N$157: J9.3, R83.2
- new net N$158: R82.1, U17.1
- new net N$159: D30.A, D34.C, K3.3, Q45.3
- new net N$160: D28.C, D29.C, D30.C, D31.C, K1.2, K2.2, K3.2, K4.2, R85.2, R86.2, R87.2
- new net N$161: D29.A, D33.C, K2.3, Q44.3
- new net N$162: R83.1, U18.1
- new net N$163: J11.2, K2.1
- new net N$164: J11.1, K2.4
- new net N$165: J11.3, K2.5
- new net N$166: J12.2, K3.1
- new net N$167: J12.1, K3.4
- new net N$168: J12.3, K3.5
- new net N$169: J13.1, K4.4
- new net N$170: J13.2, K4.1
- new net N$171: J13.3, K4.5
- new net N$172: R84.2
- new net N$173: D32.A, R84.1
- new net N$174: D34.A, R86.1
- new net N$175: D35.A, R87.1
- new net N$176: D28.A, D32.C, K1.3, Q43.3
- new net RELAY1EN: Q43.1
- new net RELAY2EN: Q44.1
- new net RELAY3EN: Q45.1
- new net RELAY4EN: Q46.1
- new net STEPPER1DIR: Q38.1, R74.2
- new net STEPPER1DIROUT: J6.3, Q38.3
- new net STEPPER1EN: Q37.1, R73.2
- new net STEPPER1ENOUT: J6.2, Q37.3
- new net STEPPER1STEP: Q39.1, R75.2
- new net STEPPER2DIR: Q41.1, R77.2
- new net STEPPER2EN: Q40.1, R76.2
- new net STEPPER2STEP: Q42.1, R78.2
- new net VBATTISENSE: F1.2@1, F1.2@2, R79.1
- net +5V: now also J6.1, J7.1
- net GND: now also J1.1, J8.4, J9.4, JP9.1, Q37.2, Q38.2, Q39.2, Q40.2, Q41.2, Q42.2, Q43.2, Q44.2, Q45.2, Q46.2, R35.1, R37.1, R39.1, R41.1, R43.1, R45.1, R47.1, R49.1, R51.1, R53.1, R55.1, R57.1, R69.1, R70.1, R71.1, R72.1, R73.1, R74.1, R75.1, R76.1, R77.1, R78.1, U14.1, U14.2, U14.3, U14.4, U15.2, U15.3, U16.2, U16.3, U17.2, U17.3, U18.2, U18.3; no longer D10.C, D11.C, D12.C, D13.C, D14.C, D15.C, D16.C, D17.C, D18.C, D19.C, D8.C, D9.C, JGND.1, JGND.2, JGND.3, JGND.4, JGND.5, JP5.1, JP6.1, JP7.1, JP8.1
- net N$100: now also D18.C, R55.2; no longer D19.A, R57.1
- net N$101: now also J1.2; no longer JBATT.1, JBATT.2, JBATT.3, JBATT.4, JBATT.5
- net N$57: now also D26.A, J5.2; no longer JP8.3
- net N$59: now also D27.A, J5.1; no longer JP8.2
- net N$61: no longer Q34.1
- net N$63: now also D25.A, J5.4; no longer JP8.5
- net N$65: now also D8.A, J2.4; no longer JP5.5, R35.2
- net N$66: now also D9.A, J2.3; no longer JP5.4, R37.2
- net N$67: now also D10.A, J2.2; no longer JP5.3, R39.2
- net N$68: now also D11.A, J2.1; no longer R41.2
- net N$69: now also D12.A, J3.4; no longer JP6.5, R43.2
- net N$70: now also D13.A, J3.3; no longer JP6.4, R45.2
- net N$71: now also D14.A, J3.2; no longer JP6.3, R47.2
- net N$72: now also D15.A, J3.1; no longer JP6.2, R49.2
- net N$73: now also D16.A, J4.4; no longer JP7.5, R51.2
- net N$74: now also D17.A, J4.3; no longer JP7.4, R53.2
- net N$75: now also D11.C, R41.2; no longer D17.A, R53.1
- net N$77: now also D12.C, R43.2; no longer D15.A, R49.1
- net N$78: now also D27.C, R72.2; no longer D14.A, R47.1
- net N$79: now also D26.C, R71.2; no longer D13.A, R45.1
- net N$80: now also D24.C, R69.2; no longer D12.A, R43.1
- net N$81: now also D25.C, R70.2; no longer D11.A, R41.1
- net N$82: now also D10.C, R39.2; no longer D10.A, R39.1
- net N$83: now also D9.C, R37.2; no longer D9.A, R37.1
- net N$84: now also D8.C, R35.2; no longer D8.A, R35.1
- net N$85: now also D24.A, J5.3; no longer JP8.4
- net N$93: now also D18.A, J4.2; no longer JP7.3, R55.2
- net N$94: now also D19.A, J4.1; no longer JP7.2, R57.2
- net N$98: now also D19.C, R57.2; no longer D18.A, R55.1
- net VBATT: now also J8.1, J9.1, R79.2; no longer F1.2@1, F1.2@2
- net VCC: now also R66.2, R67.2, R68.2, U14.8
Routing:
- net GND: track 18.4 -> 0.00 mm, vias 2 -> 0
- net SCL: track 17.9 -> 0.00 mm, vias 1 -> 0
- net SDA: track 15.2 -> 0.00 mm
- net N$4: track 11.6 -> 0.00 mm
- net N$23: track 11.6 -> 0.00 mm
- net N$18: track 11.6 -> 0.00 mm
- net N$15: track 11.6 -> 0.00 mm
- net N$9: track 10.2 -> 0.00 mm, vias 2 -> 0
- net N$38: track 10.2 -> 0.00 mm, vias 2 -> 0
- net N$25: track 10.2 -> 0.00 mm, vias 2 -> 0
- net N$17: track 10.2 -> 0.00 mm, vias 2 -> 0
- net N$26: track 7.92 -> 0.00 mm
- net N$10: track 7.92 -> 0.00 mm
- net N$39: track 7.92 -> 0.00 mm
- net N$19: track 7.92 -> 0.00 mm
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Other:
- board size 150 x 100 mm -> 200 x 150 mm

Commit message: mostly layout changes
Parts:
- removed $5_223_$_2016-03-04_22-58-43, $5_224_$_2016-03-04_22-58-43, TP1, TP2, TP3, TP4: (no value), holla:TPTHRU
- removed C10, C11, C12, C13, C14, C18, C19, C20, C21, C4, C5, C6, C7, C8, C9: .1u, holla:C0603
- removed C23: (no value), holla:C0603
- removed D4, D5, D6, D7: (no value), holla:TVS-0603
- removed J6: (no value), holla:1984633
- removed JP1, JP2, JP3, JP4: DNP, holla:PAD-JUMPER-2-NO_NO_SILK
- removed R11, R16, R17, R18, R19, R20, R21, R22, R23, R6, R7, R8, R9: 1k, holla:R0603
- removed R12, R13, R14, R15: 10k, holla:R0603
- removed R24, R25, R26, R27: 100, holla:R0603
- removed U11, U12, U9: (no value), holla:MSOP10_0.5
- removed U6, U7: (no value), holla:SO08
- added C24, C25, C26, C27, C28, C29, C30, C31, C32, C33, C34, C35, C36, C37, C38: (no value), holla:C0603
- added D36, D37: (no value), holla:LED0603
- added J10, J15, J23, J24, J25, J26, J27, J28: (no value), holla:CONN-3.81MM-KF2EDG-2
- added J16: OLED DISPLAY, holla:1X04
- added J17, J18, J19, J20, J21, J22, J31: (no value), holla:CONN-3.81MM-KF2EDG-6
- added J29, J30: (no value), holla:CONN-3.81MM-KF2EDG-3
- added J32: (no value), holla:CONN-3.81MM-KF2EDG-5
- added Q47: FDD4141, brightleaf:TO252
- added R88, R89, R92, R93, R94, R95: (no value), holla:R0603
- added R90: DNP, holla:R0603
- added R91: 0, holla:R0603
- added U19, U20: RELAY-S108T02PTH, holla:RELAY-S108T02
- added U21: IO-HC4051, holla:SO16
- added U22: (no value), holla:SO28W
- C3: value .1u -> (none)
- J11, J12, J13, J14: device holla:1984620 -> holla:CONN-3.81MM-KF2EDG-3
- J2, J3, J4, J5, J8, J9: device holla:1984633 -> holla:CONN-3.81MM-KF2EDG-4
- J7: device holla:1984633 -> holla:CONN-3.81MM-KF2EDG-5
- R10: value 1k -> 47k; device holla:R0603 -> rcl:R0402
- R4, R5: value 1k -> (none)
- R59, R63: device holla:R0603 -> holla:R1210
- U4: device holla:SO08 -> holla:SOIC8
- U5: value (none) -> AZ23C5V1; device holla:SO08 -> brightleaf:SOT-23
- moved R65 683.8 mm to (6.50, 45.8), turned to 180 degrees
- moved Q35 682.3 mm to (8.50, 25.0), turned to 180 degrees
- moved Q36 680.5 mm to (8.50, 37.5), turned to 180 degrees
- moved Q34 676.1 mm to (10.2, 45.8), turned to 180 degrees
- moved R63 669.4 mm to (13.7, 50.5), turned to 90 degrees
- moved R62 663.8 mm to (17.5, 45.8), turned to 180 degrees
- moved Q32 662.9 mm to (19.0, 25.0), turned to 180 degrees
- moved Q33 661.0 mm to (19.0, 37.5), turned to 180 degrees
- moved R72 660.9 mm to (24.0, 17.5)
- moved D27 659.0 mm to (27.0, 14.5)
- moved R64 658.0 mm to (30.0, 17.5), turned to 270 degrees
- moved D22 657.5 mm to (27.0, 16.5)
- moved D23 657.5 mm to (27.0, 18.0)
- moved Q31 656.1 mm to (21.2, 45.8), turned to 180 degrees
- moved J5 652.9 mm to (33.0, 8.00), turned to 0 degrees
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Connections:
- net N$108 renamed UART0_TX
- net N$109 renamed UART0_RX
- removed net ADC0_0: U8.4
- removed net ADC1_0: U9.4
- removed net ADC1_1: U9.5
- removed net ADC1_2: U9.6
- removed net ADC1_3: U9.7
- removed net ADC2_0: D6.1, R26.2, TP1.1, U11.4
- removed net ADC2_1: D7.1, R27.2, TP2.1, U11.5
- removed net ADC2_2: D4.1, R24.2, TP3.1, U11.6
- removed net ADC2_3: D5.1, R25.2, TP4.1, U11.7
- removed net ADC3_0: R30.2, U10.1, U12.4
- removed net ADC3_1: R33.2, U10.7, U12.5
- removed net ADC3_2: U12.6
- removed net ADC3_3: U12.7
- removed net N$10: R10.2, R11.2, R15.1, U7.2
- removed net N$11: U7.3
- removed net N$12: JP4.2, R10.1
- removed net N$13: C11.1, R20.2, U4.6
- removed net N$14: JP3.2, R8.1
- removed net N$15: C7.1, R24.1, U4.5, U4.7
- removed net N$16: C7.2, R16.2, R20.1
- removed net N$17: R12.2, R16.1, U4.1
- removed net N$18: C9.1, R26.1, U6.5, U6.7
- removed net N$19: R12.1, R4.2, R5.2, U4.2
- removed net N$20: U4.3
- removed net N$21: JP1.2, R4.1
- removed net N$22: C12.1, R21.2, U5.6
- removed net N$23: C8.1, R25.1, U5.5, U5.7
- removed net N$24: C8.2, R17.2, R21.1
- removed net N$25: R13.2, R17.1, U5.1
- removed net N$26: R13.1, R6.2, R7.2, U5.2
- removed net N$27: U5.3
- removed net N$28: JP2.2, R6.1
- removed net N$38: R14.2, R18.1, U6.1
- removed net N$39: R14.1, R8.2, R9.2, U6.2
- removed net N$55: U6.3
- removed net SUPPLY: C1.1, U2.8
- removed net VCC: C18.1, C19.1, C2.1, C20.1, C21.1, C22.1, C23.1, R66.2, R67.2, R68.2, U11.8, U12.8, U13.1, U13.28, U13.3, U13.5, U14.8, U3.8, U8.8, U9.1, U9.8
- new net +3V3: J22.1, J22.2, J22.3, J22.4, J22.5, J22.6, PCB1.P$1, R66.2, R67.2, R68.2, U14.8
- new net C_24IN: F1.2@1, F1.2@2, Q47.3
- new net INPUTINTERRUPT: U22.19
- new net N$108: C26.1, J17.3, U22.5
- new net N$109: C27.1, J17.4, U22.6
- new net N$177: J10.2, U19.2
- new net N$178: J15.1, U20.1
- new net N$179: J15.2, U20.2
- new net N$180: D36.C, R88.2
- new net N$181: D37.C, R89.2
- new net N$182: D36.A, U19.4
- new net N$183: D37.A, U20.4
- new net N$184: C34.1, J26.2, U21.1
- new net N$185: C35.1, J25.2, U21.5
- new net N$186: C36.1, J24.2, U21.2
- new net N$187: C37.1, J23.2, U21.4
- new net N$76: J10.1, U19.1
- new net RELAY0EN: Q43.1, U22.21
- new net RELAY5EN: R89.1, U22.26
- new net SENSORS0: U21.11
- new net SENSORS1: U21.10
- new net SENSORS2: U21.9
- net +5V: now also C1.1, C2.1, C22.1, C3.1, C38.1, J16.2, J20.1, J20.2, J20.3, J20.4, J20.5, J20.6, J29.3, J30.3, J31.6, J32.5, J7.5, PCB1.P$2, PCB1.P$4, R90.2, R92.2, R93.2, R94.2, R95.2, U13.24, U13.28, U19.3, U2.8, U20.3, U21.16, U22.18, U22.9, U3.5, U3.8, U4.5, U8.8; no longer J6.1, J7.1
- net ADC0_1: now also R30.2, U10.1
- net ADC0_2: now also R33.2, U10.7
- net AGND: no longer C11.2, C12.2, C13.2, C14.2, C15.2, C16.2, C17.2, C3.2, C4.2, C5.2, C6.2, D4.2, D5.2, D6.2, D7.2, JP1.1, JP2.1, JP3.1, JP4.1, R11.1, R5.1, R7.1, R9.1, U10.4, U4.4, U5.4, U6.4, U7.4
- net AVCC: no longer C3.1, C4.1, C5.1, C6.1, U4.8, U5.8, U6.8, U7.8
- net GND: now also C15.2, C16.2, C17.2, C24.2, C25.2, C26.2, C27.2, C28.2, C29.2, C3.2, C30.2, C31.2, C32.2, C33.2, C34.2, C35.2, C36.2, C37.2, C38.2, J16.1, J18.1, J18.2, J18.3, J18.4, J18.5, J18.6, J21.1, J21.2, J21.3, J21.4, J21.5, J21.6, J23.1, J24.1, J25.1, J26.1, J27.1, J28.1, J29.1, J30.1, J31.1, J32.1, J7.1, PCB1.P$14, PCB1.P$20, PCB1.P$25, PCB1.P$30, PCB1.P$34, PCB1.P$39, PCB1.P$6, PCB1.P$9, R10.1, R5.1, U10.4, U13.1, U13.3, U13.5, U21.6, U21.7, U21.8, U22.10, U22.15, U22.16, U22.17, U4.1, U4.2, U4.6; no longer C18.2, C19.2, C20.2, C21.2, C23.2, U11.3, U12.3, U13.24, U3.5, U9.3
- net N$102: now also C24.1, J17.1, U22.3; no longer PCB1.P$2
- net N$103: now also C25.1, J17.2, U22.4; no longer PCB1.P$4
- net N$106: now also PCB1.P$7; no longer PCB1.P$6
- net N$111: now also C28.1, J17.5, U22.7; no longer PCB1.P$14
- net N$114: now also C29.1, J17.6, U22.8; no longer PCB1.P$20
- net N$118: now also U21.3, U8.4; no longer PCB1.P$30
- net N$120: now also C30.1, J30.2, R92.1, U21.13; no longer PCB1.P$34
- net N$124: now also C31.1, J29.2, R93.1, U21.14; no longer PCB1.P$39
- net N$130: now also C32.1, R4.1, R5.2, R94.1, U21.15; no longer PCB1.P$25
- net N$138: now also C33.1, J27.2, R95.1, U21.12; no longer PCB1.P$9
- net N$151: now also J32.2; no longer J6.4
- net N$152: now also J7.4; no longer J7.2
- net N$154: now also J7.2; no longer J7.4
- net N$172: now also R90.1, R91.1
- net N$2: now also J28.2, R4.2; no longer C14.1, R23.2, U7.6
- net N$4: now also Q47.1, R10.2, U5.1; no longer C10.1, R27.1, U7.5, U7.7
- net N$6: now also J31.5, U22.27; no longer C10.2, R19.2, R23.1
- net N$7: now also J31.4, U22.28; no longer C9.2, R18.2, R22.1
- net N$8: now also J31.3, U22.1; no longer C13.1, R22.2, U6.6
- net N$9: now also J31.2, U22.2; no longer R15.2, R19.1, U7.1
- net RELAY1EN: now also Q44.1, U22.22; no longer Q43.1
- net RELAY2EN: now also Q45.1, U22.23; no longer Q44.1
- net RELAY3EN: now also Q46.1, U22.24; no longer Q45.1
- net RELAY4EN: now also R88.1, U22.25; no longer Q46.1
- net SCL: now also J16.3, PCB1.P$5, U22.12, U4.4; no longer $5_224_$_2016-03-04_22-58-43.1, U11.10, U12.1, U12.10, U9.10
- net SDA: now also J16.4, PCB1.P$3, U22.13, U4.3; no longer $5_223_$_2016-03-04_22-58-43.1, U11.1, U11.9, U12.9, U9.9
- net STEPPER1DIROUT: now also J32.3; no longer J6.3
- net STEPPER1ENOUT: now also J32.4; no longer J6.2
- net VBATT: now also J19.1, J19.2, J19.3, J19.4, J19.5, J19.6, R91.2, U4.7
- net VBATTISENSE: now also Q47.2, U4.8, U5.2, U5.3; no longer F1.2@1, F1.2@2
Routing:
- net N$59: track 0.00 -> 63.1 mm, vias 0 -> 6
- net N$67: track 0.00 -> 62.4 mm, vias 0 -> 6
- net VBATT: track 0.00 -> 61.3 mm, vias 0 -> 84
- net N$69: track 0.00 -> 58.1 mm, vias 0 -> 6
- net N$73: track 0.00 -> 57.6 mm, vias 0 -> 6
- net N$93: track 0.00 -> 57.4 mm, vias 0 -> 6
- net N$57: track 0.00 -> 56.9 mm, vias 0 -> 6
- net N$71: track 0.00 -> 55.9 mm, vias 0 -> 6
- net N$85: track 0.00 -> 54.1 mm, vias 0 -> 6
- net N$65: track 5.24 -> 58.6 mm, vias 0 -> 6
- net N$63: track 0.00 -> 52.0 mm, vias 0 -> 6
- net N$74: track 0.00 -> 29.6 mm, vias 0 -> 6
- net N$70: track 0.00 -> 29.6 mm, vias 0 -> 6
- net N$66: track 0.00 -> 29.4 mm, vias 0 -> 6
- net N$94: track 0.00 -> 28.4 mm, vias 0 -> 6
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- added copper zone on layer 1, net MOTORA_SENSE
- added copper zone on layer 16, net MOTORA_SENSE
- added copper zone on layer 1, net MOTORB_SENSE
- added copper zone on layer 16, net MOTORB_SENSE
- added copper zone on layer 1, net VBATT

Commit message: parts placed
Parts:
- removed J18, J20, J22: (no value), holla:CONN-3.81MM-KF2EDG-6
- added C4, C5: .1u, holla:C0603
- added D4: (no value), holla:DO-214AC(SMA)
- added J6: (no value), holla:CONN-3.81MM-KF2EDG-5
- added R11: 120, holla:R0603
- added R12, R13, R14, R15, R6, R7, R8, R9: (no value), holla:R0603
- added S1, S2, S3, S4: (no value), holla:TACTILE-SWITCH-6MMX3.5MM
- added U6: (no value), holla:DISP-I2C-4PIN-0.96
- added U7: (no value), holla:SO14
- J16: value OLED DISPLAY -> (none); device holla:1X04 -> holla:1X02
- moved C3 350.7 mm to (16.0, 63.0)
- moved U4 345.8 mm to (21.5, 47.5), turned to 0 degrees
- moved J32 329.5 mm to (65.5, 78.5), turned to 0 degrees
- moved C37 315.0 mm to (14.0, 91.0), turned to 0 degrees
- moved C36 302.8 mm to (23.5, 91.0), turned to 0 degrees
- moved J7 300.9 mm to (87.0, 78.5), turned to 0 degrees
- moved R5 300.6 mm to (59.0, 90.5)
- moved R4 299.5 mm to (56.0, 91.0), turned to 180 degrees
- moved C38 291.6 mm to (56.0, 61.0)
- moved C35 290.6 mm to (33.0, 91.0), turned to 0 degrees
- moved J27 288.2 mm to (49.5, 97.0), turned to 180 degrees
- moved J28 287.8 mm to (59.0, 97.0), turned to 180 degrees
- moved C34 278.5 mm to (42.5, 91.0), turned to 0 degrees
- moved J31 238.8 mm to (128.5, 97.0), turned to 180 degrees
- moved J1 236.5 mm to (8.00, 86.5), turned to 270 degrees
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Connections:
- new net N$10: U7.5
- new net N$11: U7.2
- new net N$12: U7.4
- new net N$13: J6.2, R11.2, U7.12
- new net N$14: J6.3, R11.1, U7.11
- new net N$15: J6.4, U7.9
- new net N$16: J6.5, U7.10
- new net N$17: J16.2, J6.1
- new net N$19: U7.3
- new net N$21: R15.1, S1.P$2
- new net N$22: R14.1, S2.P$2
- new net N$23: R13.1, S3.P$2
- new net N$24: R12.1, S4.P$2
- net +3V3: now also C5.1, R12.2, R13.2, R14.2, R15.2, U7.1; no longer J22.1, J22.2, J22.3, J22.4, J22.5, J22.6
- net +5V: now also C4.1, J19.4, J19.5, J19.6, R6.2, R7.2, R8.2, R9.2, U6.VCC, U7.14; no longer J16.2, J20.1, J20.2, J20.3, J20.4, J20.5, J20.6
- net GND: now also C4.2, C5.2, D4.A, S1.P$1, S2.P$1, S3.P$1, S4.P$1, U6.GND, U7.6, U7.8; no longer J18.1, J18.2, J18.3, J18.4, J18.5, J18.6
- net N$184: now also R6.1
- net N$185: now also R7.1
- net N$186: now also R8.1
- net N$187: now also R9.1
- net N$6: now also J31.2; no longer J31.5
- net N$7: now also J31.5, U22.2; no longer J31.4, U22.28
- net N$8: now also J31.4; no longer J31.3
- net N$9: now also J31.3, U22.28; no longer J31.2, U22.2
- net SCL: now also U6.SCL; no longer J16.3
- net SDA: now also U6.SDA; no longer J16.4
- net VBATT: now also D4.C; no longer J19.4, J19.5, J19.6
Routing:
- net N$47: track 0.00 -> 56.5 mm, vias 0 -> 2
- net N$49: track 0.00 -> 48.0 mm, vias 0 -> 2
- net N$187: track 0.00 -> 47.1 mm
- net N$51: track 0.00 -> 40.1 mm, vias 0 -> 2
- net N$1: track 0.00 -> 38.0 mm, vias 0 -> 2
- net N$53: track 0.00 -> 36.4 mm
- net N$186: track 0.00 -> 35.9 mm
- net N$185: track 0.00 -> 33.7 mm, vias 0 -> 1
- net N$48: track 0.00 -> 30.1 mm, vias 0 -> 2
- net N$56: track 0.00 -> 24.1 mm
- net N$91: track 0.00 -> 23.6 mm
- net N$50: track 0.00 -> 21.9 mm, vias 0 -> 2
- net N$138: track 0.00 -> 19.8 mm
- net N$130: track 0.00 -> 18.1 mm
- net N$118: track 0.00 -> 16.6 mm
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Other:
- board size 200 x 150 mm -> 200 x 100 mm
