File: board/tex.brd (EAGLE design)
At the start: 200 x 100 mm, 270 parts, among them K1 HLS8L-DC5V-S-C, K2 HLS8L-DC5V-S-C, K3 HLS8L-DC5V-S-C, K4 HLS8L-DC5V-S-C, Q47 FDD4141, U14 24LC32A, U15 OPTO-LTV817, U16 OPTO-LTV817, U17 OPTO-LTV817, U18 OPTO-LTV817, U19 RELAY-S108T02PTH, U20 RELAY-S108T02PTH, U21 IO-HC4051, U5 AZ23C5V1, Y1 32.768KHz

Commit message: board file submission
Parts:
- removed C35, C38: (no value), holla:C0603
- removed D0, D37: (no value), holla:LED0603
- removed J31: (no value), holla:CONN-3.81MM-KF2EDG-6
- removed J32: (no value), holla:CONN-3.81MM-KF2EDG-5
- removed JP9: DNP, holla:PAD-JUMPER-2-NO_NO_SILK
- removed R0: (no value), holla:R0603
- removed R95: 120, holla:R0603
- removed S0: (no value), holla:TACTILE-SWITCH-6MMX3.5MM
- removed U21: IO-HC4051, holla:SO16
- removed U22: (no value), holla:SO28W
- added C13, C14: .1u, holla:C0603
- added D3, D7: (no value), holla:LED0603
- added J20: (no value), holla:CONN-OSTT702
- added J22: (no value), holla:CONN-3.81MM-KF2EDG-2
- added JP3: FIDUCIALUFIDUCIAL, holla:MICRO-FIDUCIAL
- added R14, R15: (no value), holla:R0603
- added S2: (no value), holla:TACTILE-SWITCH-6MMX3.5MM
- added U12: OPTO-LTV817, holla:LTV817
- added U9: (no value), holla:DCDC-LM2577-BOARD
- C10, C3: value (none) -> .1u
- C11, C15, C17, C2: value .1u -> (none)
- D21, D22, D23, D24: device holla:LED0603 -> holla:SOD-523
- D28, D29, D30: device holla:SOD-523 -> holla:LED0603
- D31: device holla:SOD-523 -> holla:DO-214AC(SMA)
- D35, D36: device holla:LED0603 -> holla:SOD-323
- D4: device holla:DO-214AC(SMA) -> holla:LED0603
- D5, D6: device holla:SOD-323 -> holla:LED0603
- J1: device holla:CONN-OSTT702 -> holla:CONN-3.81MM-KF2EDG-4
- J10, J27, J28: device holla:CONN-3.81MM-KF2EDG-2 -> holla:CONN-3.81MM-KF2EDG-3
- J11: device holla:CONN-3.81MM-KF2EDG-3 -> holla:1X04
- J12: device holla:CONN-3.81MM-KF2EDG-3 -> holla:1X02
- J13: device holla:CONN-3.81MM-KF2EDG-3 -> holla:CONN-3.81MM-KF2EDG-5
- J14: device holla:CONN-3.81MM-KF2EDG-3 -> holla:CONN-3.81MM-KF2EDG-4
- J15: device holla:CONN-3.81MM-KF2EDG-2 -> holla:CONN-3.81MM-KF2EDG-4
- J16: device holla:1X02 -> holla:CONN-3.81MM-KF2EDG-6
- J17: device holla:CONN-3.81MM-KF2EDG-6 -> holla:CONN-3.81MM-KF2EDG-5
- J18: device holla:1X04 -> holla:CONN-3.81MM-KF2EDG-5
- J21: device holla:CONN-3.81MM-KF2EDG-6 -> holla:CONN-3.81MM-KF2EDG-2
- J29, J30: device holla:CONN-3.81MM-KF2EDG-3 -> holla:CONN-3.81MM-KF2EDG-6
- J5: device holla:CONN-3.81MM-KF2EDG-4 -> holla:CONN-3.81MM-KF2EDG-2
- J6: device holla:CONN-3.81MM-KF2EDG-5 -> holla:CONN-3.81MM-KF2EDG-2
- J7: device holla:CONN-3.81MM-KF2EDG-5 -> holla:CONN-3.81MM-KF2EDG-3
- J8, J9: device holla:CONN-3.81MM-KF2EDG-4 -> holla:CONN-3.81MM-KF2EDG-3
- JP2: value FIDUCIALUFIDUCIAL -> DNP; device holla:MICRO-FIDUCIAL -> holla:PAD-JUMPER-2-NO_NO_SILK
- Q1, Q21, Q23, Q25, Q28, Q3, Q5, Q7, Q9: device holla:SOT23-3 -> holla:TO252
- Q12, Q14, Q16, Q18, Q20, Q32, Q33, Q35, Q36: device holla:TO252 -> holla:SOT23-3
- Q41: value (none) -> FDD4141; device holla:SOT23-3 -> brightleaf:TO252
- Q47: value FDD4141 -> (none); device brightleaf:TO252 -> holla:SOT23-3
- R10: value 47k -> (none)
- R11, R93, R94: value 120 -> (none)
- R19: value (none) -> 0
- R20, R21, R29, R31, R32, R66: value 1k -> (none)
- R22, R91: value 0 -> (none)
- R23, R90: value DNP -> (none)
- R24, R30: value 10k -> (none)
- R28: value 1k -> DNP
- R33: value 10k -> (none); device holla:R0603 -> holla:R1210
- R34, R51: device holla:R0603 -> holla:R1210
- R39, R40, R52: value (none) -> 120
- R43: value (none) -> 47k
- R44, R55, R56, R57, R71, R72, R77: value (none) -> 1k
- R53, R54, R69: value (none) -> 10k
- R59: device holla:R1210 -> holla:R0603
- R63: value (none) -> 0; device holla:R1210 -> holla:R0603
- R67, R68: value 3.9k -> (none)
- R70: value (none) -> DNP
- R73, R74: value (none) -> 3.9k
- R79: value (none) -> 120; device holla:R1210 -> holla:R0603
- U1: value (none) -> RELAY-S108T02PTH; device holla:DCDC-LM2577-BOARD -> holla:RELAY-S108T02
- U10: device holla:SO08 -> holla:MSOP10_0.5
- U13: value (none) -> OPTO-LTV817; device holla:TSSOP28 -> holla:LTV817
- U14: value 24LC32A -> OPTO-LTV817; device holla:SO08 -> holla:LTV817
- U16: value OPTO-LTV817 -> (none); device holla:LTV817 -> holla:SO28W
- U17: value OPTO-LTV817 -> 24LC32A; device holla:LTV817 -> holla:SO08
- U18: value OPTO-LTV817 -> IO-HC4051; device holla:LTV817 -> holla:SO16
- U19: value RELAY-S108T02PTH -> (none); device holla:RELAY-S108T02 -> holla:SO08
- U2: value (none) -> RELAY-S108T02PTH; device holla:SO08 -> holla:RELAY-S108T02
- U20: value RELAY-S108T02PTH -> (none); device holla:RELAY-S108T02 -> holla:DISP-I2C-4PIN-0.96
- U3: device holla:SO08 -> holla:SO14
- U4: value (none) -> AZ23C5V1; device holla:SOIC8 -> brightleaf:SOT-23
- U5: value AZ23C5V1 -> (none); device brightleaf:SOT-23 -> holla:TSSOP28
- U6: device holla:DISP-I2C-4PIN-0.96 -> holla:SO08
- U7: device holla:SO14 -> holla:SOIC8
- U8: device holla:MSOP10_0.5 -> holla:SO08
- moved R79 168.8 mm to (190.0, 80.5), turned to 180 degrees
- moved R62 163.7 mm to (176.5, 67.5), turned to 0 degrees
- moved D1 158.7 mm to (24.5, 9.50), turned to 90 degrees
- moved D2 158.2 mm to (28.5, 9.50)
- moved C16 157.8 mm to (190.0, 84.0)
- moved C8 156.7 mm to (198.0, 59.2), turned to 90 degrees
- moved D24 155.2 mm to (186.5, 28.5), turned to 180 degrees
- moved R61 152.4 mm to (173.0, 67.5), turned to 0 degrees
- moved C12 148.5 mm to (48.5, 73.0), turned to 180 degrees
- moved U8 147.6 mm to (194.0, 61.0), turned to 180 degrees
- moved R32 147.0 mm to (182.0, 29.5), turned to 270 degrees
- moved R1 145.9 mm to (39.4, 8.89), turned to 90 degrees
- moved D23 145.8 mm to (169.5, 28.5), turned to 180 degrees
- moved C11 144.6 mm to (44.5, 72.9), turned to 180 degrees
- moved R60 141.4 mm to (169.5, 67.5), turned to 0 degrees
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- renumbered B1 to B100, C30 to C19, C31 to C18, C34 to C23, C36 to C21, C37 to C20
Connections:
- net +3V3: now also C1.1, R39.2, R40.2, R41.2, R42.2, R73.2, R74.2, R77.2, U17.8, U3.1; no longer C5.1, R12.2, R13.2, R66.2, R67.2, R68.2, R93.2, R94.2, U14.8, U7.1
- net +5V: now also C16.1, C6.1, C8.1, J11.2, J16.4, J16.5, J16.6, J17.5, J18.5, J27.3, J28.3, J30.6, R28.2, R78.1, R79.2, U1.3, U16.18, U16.9, U19.8, U2.3, U20.VCC, U3.14, U5.24, U5.28, U7.5, U8.5, U8.8, U9.OUT+; no longer C1.1, C22.1, C4.1, J18.2, J19.4, J19.5, J19.6, J29.3, J30.3, J31.6, J32.5, J7.5, R3.1, R90.2, R95.2, U1.OUT+, U13.24, U13.28, U19.3, U2.8, U20.3, U22.18, U22.9, U3.5, U3.8, U4.5, U6.VCC, U7.14
- net ADC0_1: now also R53.2, U10.5, U6.1; no longer R30.2, U10.1, U8.5
- net ADC0_2: now also R54.2, U10.6, U6.7; no longer R33.2, U10.7, U8.6
- net ADCALERT: now also U10.2; no longer U8.2
- net AGND: now also C11.2, C12.2, C22.2, C4.2, C5.2, J21.1, J22.1, R55.1, R56.1, R59.1, R64.2, R70.1, R71.1, R75.1, R87.1, R89.1, U10.1, U10.3, U10.7, U18.6, U18.7, U18.8, U6.4; no longer C16.2, C35.2, C38.2, C6.2, C8.2, J29.1, J30.1, R17.1, R19.1, R21.1, R23.1, R25.2, R27.1, R28.1, R31.1, R5.1, U10.4, U21.6, U21.7, U21.8, U8.1, U8.3, U8.7
- net AVCC: now also C15.1, C5.1, C7.1, R78.2, R90.2, R91.2, R93.2, R94.2, U18.16, U6.8; no longer C16.1, C38.1, C8.1, R3.2, R6.2, R7.2, R8.2, R9.2, U21.16, U8.8
- net D0: now also R60.2; no longer R0.2
- net D1: now also R61.2; no longer R1.2
- net D2: now also R62.2; no longer R2.2
- net DCMOTORAENCA: now also U14.4; no longer U15.4
- net DCMOTORAENCB: now also U15.4; no longer U16.4
- net DCMOTORBENCA: now also U12.4; no longer U17.4
- net DCMOTORBENCB: now also U13.4; no longer U18.4
- net GND: now also C13.2, C14.2, C16.2, C6.2, C8.2, D31.A, D32.C, D33.C, D34.C, J11.1, J12.1, J14.4, J15.4, J17.1, J19.1, J19.2, J19.3, J19.4, J19.5, J19.6, J20.1, J30.1, JP2.1, Q12.2, Q14.2, Q16.2, Q18.2, Q20.2, Q32.2, Q33.2, Q35.2, Q36.2, Q47.2, R1.1, R10.1, R11.1, R12.1, R13.1, R14.1, R16.1, R17.1, R2.1, R3.1, R33.2, R34.2, R4.1, R43.2, R5.1, R6.1, R64.1, R7.1, R8.1, R80.1, R81.1, R82.1, R83.1, R84.1, R85.1, R9.1, S2.P$1, U12.2, U12.3, U16.10, U16.15, U16.16, U16.17, U17.1, U17.4, U19.4, U20.GND, U3.8, U5.1, U5.14, U5.2, U5.23, U5.25, U5.3, U5.4, U5.5, U7.1, U7.2, U8.4, U8.6, U8.7, U9.IN-, U9.OUT-; no longer C11.2, C12.2, C22.2, C4.2, C5.2, D0.C, D1.C, D2.C, D4.A, J1.1, J16.1, J21.1, J21.2, J21.3, J21.4, J21.5, J21.6, J31.1, J32.1, J7.1, J8.4, J9.4, JP9.1, Q1.2, Q21.2, Q23.2, Q25.2, Q28.2, Q3.2, Q41.2, Q5.2, Q7.2, Q9.2, R10.2, R25.1, R35.1, R37.1, R39.1, R41.1, R43.1, R45.1, R47.1, R49.1, R51.1, R53.1, R55.1, R57.1, R59.2, R63.2, R69.1, R70.1, R71.1, R72.1, R73.1, R74.1, R75.1, R76.1, R77.1, R78.1, S0.P$1, U1.IN-, U1.OUT-, U13.1, U13.14, U13.23, U13.25, U13.4, U13.5, U14.1, U14.4, U16.2, U16.3, U18.2, U18.3, U2.4, U22.10, U22.15, U22.16, U22.17, U3.4, U3.7, U4.1, U4.2, U4.6, U6.GND, U7.8
- net GND4: now also D21.A, D27.C, K2.3, Q18.3; no longer D31.A, D35.C, K4.3, Q46.3
- net ID_SC: now also R73.1, U17.6; no longer R67.1, U14.6
- net ID_SD: now also R74.1, U17.5; no longer R68.1, U14.5
- net INPUTINTERRUPT: now also U16.19; no longer U22.19
- net MOTORA_SENSE: now also Q1.2, Q2.2, R33.1, R44.1; no longer Q32.2, Q35.2, R29.1, R63.1
- net MOTORB_SENSE: now also Q3.2, Q4.2, R34.1, R57.1; no longer Q26.2, Q29.2, R32.1, R59.1
- net N$1: now also Q40.1, U5.6; no longer Q1.1, U13.6
- net N$100: now also D6.C, R3.2; no longer D18.C, R55.2
- net N$101: now also J20.2; no longer J1.2
- net N$102: now also C29.1, J29.1, U16.3; no longer C24.1, J17.1, U22.3
- net N$103: now also C28.1, J29.2, U16.4; no longer C25.1, J17.2, U22.4
- net N$104: now also JP2.2, R77.1, U17.7; no longer JP9.2, R66.1, U14.7
- net N$105: now also R53.1, R56.2, U6.2; no longer R28.2, R30.1, U10.2
- net N$107: now also C9.1, R57.2, U6.5; no longer C17.1, R32.2, U10.5
- net N$108: now also C27.1, J29.3, U16.5; no longer C26.1, J17.3, U22.5
- net N$109: now also C26.1, J29.4, U16.6; no longer C27.1, J17.4, U22.6
- net N$111: now also C25.1, J29.5, U16.7; no longer C28.1, J17.5, U22.7
- net N$114: now also C24.1, J29.6, U16.8; no longer C29.1, J17.6, U22.8
- net N$118: now also U19.3; no longer U2.3
- net N$120: now also J28.2, R90.1, U18.13; no longer J30.2, R92.1, U21.13
- net N$124: now also R88.1, R89.2, U18.14; no longer R18.1, R19.2, U21.14
- net N$13: now also J13.2, R52.2, U3.12; no longer J6.2, R11.2, U7.12
- net N$130: now also C17.1, R86.1, R87.2, U18.15; no longer C6.1, R4.1, R5.2, U21.15
- net N$138: now also C11.1, R75.2, R76.1; no longer C7.1, R16.1, R17.2
- net N$139: now also D7.C, R4.2; no longer D17.C, R53.2
- net N$14: now also J13.3, R52.1, U3.11; no longer J6.3, R11.1, U7.11
- net N$140: now also D8.C, R5.2; no longer D16.C, R51.2
- net N$141: now also D9.C, R6.2; no longer D15.C, R49.2
- net N$142: now also D10.C, R7.2; no longer D14.C, R47.2
- net N$143: now also J10.2, K4.1; no longer J14.2, K1.1
- net N$144: now also J10.1, K4.4; no longer J14.1, K1.4
- net N$145: now also J10.3, K4.5; no longer J14.3, K1.5
- net N$146: now also D11.C, R8.2; no longer D13.C, R45.2
- net N$147: now also D29.A, R31.1; no longer D33.A, R85.1
- net N$148: now also R67.1, U14.1; no longer R80.1, U15.1
- net N$149: now also J15.3, R68.2; no longer J8.3, R81.2
- net N$15: now also J13.4, U3.9; no longer J6.4, U7.9
- net N$150: now also J15.2, R67.2; no longer J8.2, R80.2
- net N$151: now also J17.2, Q42.3; no longer J32.2, Q39.3
- net N$152: now also J18.4, Q47.3; no longer J7.4, Q40.3
- net N$153: now also J18.3, Q46.3; no longer J7.3, Q41.3
- net N$154: now also J18.2, Q45.3; no longer J7.2, Q42.3
- net N$155: now also R68.1, U15.1; no longer R81.1, U16.1
- net N$156: now also J14.2, R65.2; no longer J9.2, R82.2
- net N$157: now also J14.3, R66.2; no longer J9.3, R83.2
- net N$158: now also R65.1, U12.1; no longer R82.1, U17.1
- net N$159: now also D22.A, D28.C, K1.3, Q19.3; no longer D30.A, D34.C, K3.3, Q45.3
- net N$16: now also J13.5, U3.10; no longer J6.5, U7.10
- net N$161: now also D23.A, D29.C, K3.3, Q17.3; no longer D29.A, D33.C, K2.3, Q44.3
- net N$162: now also R66.1, U13.1; no longer R83.1, U18.1
- net N$163: now also J9.2, K3.1; no longer J11.2, K2.1
- net N$164: now also J9.1, K3.4; no longer J11.1, K2.4
- net N$165: now also J9.3, K3.5; no longer J11.3, K2.5
- net N$166: now also J8.2, K1.1; no longer J12.2, K3.1
- net N$167: now also J8.1, K1.4; no longer J12.1, K3.4
- net N$168: now also J8.3, K1.5; no longer J12.3, K3.5
- net N$169: now also J7.1, K2.4; no longer J13.1, K4.4
- net N$17: now also J12.2, J13.1; no longer J16.2, J6.1
- net N$170: now also J7.2, K2.1; no longer J13.2, K4.1
- net N$171: now also J7.3, K2.5; no longer J13.3, K4.5
- net N$172: now also D21.C, D22.C, D23.C, D24.C, R19.1, R28.1, R29.2, R30.2, R31.2, R32.2; no longer D28.C, D29.C, D30.C, D31.C, R84.2, R85.2, R86.2, R87.2, R90.1, R91.1
- net N$173: now also D30.A, R32.1; no longer D32.A, R84.1
- net N$174: now also D28.A, R30.1; no longer D34.A, R86.1
- net N$175: now also D27.A, R29.1; no longer D35.A, R87.1
- net N$176: now also D24.A, D30.C, K4.3, Q20.3; no longer D28.A, D32.C, K1.3, Q43.3
- net N$177: now also J6.2, U2.2; no longer J10.2, U19.2
- net N$178: now also J5.1, U1.1; no longer J15.1, U20.1
- net N$179: now also J5.2, U1.2; no longer J15.2, U20.2
- net N$180: now also D26.C, R26.2; no longer D36.C, R88.2
- net N$181: now also D25.C, R25.2; no longer D37.C, R89.2
- net N$182: now also D26.A, U2.4; no longer D36.A, U19.4
- net N$183: now also D25.A, U1.4; no longer D37.A, U20.4
- net N$184: now also J24.2, R94.1, U18.1; no longer J26.2, R6.1, U21.1
- net N$185: now also C22.1, J23.2, R93.1, U18.5; no longer C35.1, J25.2, R7.1, U21.5
- net N$186: now also J22.2, R92.1, U18.2; no longer J24.2, R8.1, U21.2
- net N$187: now also J21.2, R91.1, U18.4; no longer J23.2, R9.1, U21.4
- net N$188: now also R58.2, R63.2; no longer R22.2, R26.2
- net N$189: now also R72.1, U18.3; no longer R20.1, U21.3
- net N$190: now also R58.1, R59.2, U10.4; no longer R26.1, R27.2, U8.4
- net N$191: now also R69.2, U18.12; no longer R24.2, U21.12
- net N$192: now also R79.1, U19.7; no longer R95.1, U2.7
- net N$194: now also Q41.3; no longer Q47.3
- net N$2: now also D35.C, R86.2; no longer D5.C, R4.2
- net N$20: now also D35.A, J26.2; no longer D5.A, J28.2
- net N$25: now also D36.C, R76.2; no longer D6.C, R16.2
- net N$26: now also D36.A, J25.2; no longer D6.A, J27.2
- net N$27: now also J27.2, R88.2; no longer J29.2, R18.2
- net N$29: now also D32.A, R60.1; no longer D0.A, R0.1
- net N$3: now also C13.1, U19.1; no longer C11.1, U2.1
- net N$30: now also D33.A, R61.1; no longer D1.A, R1.1
- net N$31: now also D34.A, R62.1; no longer D2.A, R2.1
- net N$35: now also Q12.3, Q6.1, R20.1; no longer Q19.3, Q20.1, R52.1
- net N$36: now also Q26.1, Q36.3, R45.1; no longer Q17.3, Q18.1, R50.1
- net N$37: now also Q13.3, Q7.1, R21.1; no longer Q15.3, Q16.1, R48.1
- net N$38: now also R63.1, R70.2; no longer R22.1, R23.2
- net N$39: now also R69.1, R71.2; no longer R21.2, R24.1
- net N$4: now also Q41.1, R43.1, U4.1; no longer Q47.1, R10.1, U5.1
- net N$40: now also Q27.1, Q37.3, R47.1; no longer Q13.3, Q14.1, R46.1
- net N$41: now also Q14.3, Q8.1, R22.1; no longer Q11.3, Q12.1, R44.1
- net N$42: now also Q28.1, Q38.3, R48.1; no longer Q10.1, Q9.3, R42.1
- net N$43: now also Q15.3, Q9.1, R23.1; no longer Q7.3, Q8.1, R40.1
- net N$44: now also Q29.1, Q39.3, R49.1; no longer Q5.3, Q6.1, R38.1
- net N$45: now also Q10.1, Q16.3, R24.1; no longer Q3.3, Q4.1, R36.1
- net N$46: now also Q30.1, Q40.3, R50.1; no longer Q1.3, Q2.1, R34.1
- net N$47: now also Q16.1, U5.7; no longer Q3.1, U13.7
- net N$48: now also Q39.1, U5.8; no longer Q5.1, U13.8
- net N$49: now also Q15.1, U5.9; no longer Q7.1, U13.9
- net N$5: now also C14.1, U19.2; no longer C12.1, U2.2
- net N$50: now also Q38.1, U5.10; no longer Q9.1, U13.10
- net N$51: now also Q14.1, U5.11; no longer Q11.1, U13.11
- net N$52: now also Q37.1, U5.12; no longer Q13.1, U13.12
- net N$53: now also Q13.1, U5.13; no longer Q15.1, U13.13
- net N$54: now also Q36.1, U5.15; no longer Q17.1, U13.15
- net N$55: now also C12.1, R72.2; no longer C9.1, R20.2
- net N$56: now also Q12.1, U5.16; no longer Q19.1, U13.16
- net N$57: now also D2.A, J1.2, Q2.3, Q22.3, R15.2; no longer D26.A, J5.2, Q32.3, Q33.3, R64.2
- net N$58: now also Q2.1, Q22.1, Q33.3, R37.1; no longer Q31.3, Q32.1, Q33.1, R62.1
- net N$59: now also D1.A, D17.C, D19.A, J1.1, Q1.3, Q21.3; no longer D22.C, D23.A, D27.A, J5.1, Q35.3, Q36.3
- net N$6: now also J30.2, U16.27; no longer J31.2, U22.27
- net N$60: now also Q1.1, Q21.1, Q32.3, R36.1; no longer Q34.3, Q35.1, Q36.1, R65.1
- net N$61: now also Q32.1, U5.22; no longer Q34.1, U13.22
- net N$62: now also Q33.1, U5.21; no longer Q31.1, U13.21
- net N$63: now also D4.A, J1.4, Q24.3, Q4.3, R18.2; no longer D25.A, J5.4, Q26.3, Q27.3, R60.2
- net N$64: now also Q24.1, Q31.3, Q4.1, R35.1; no longer Q25.3, Q26.1, Q27.1, R58.1
- net N$65: now also D16.A, J4.4, Q30.3; no longer D8.A, J2.4, Q2.3
- net N$66: now also D15.A, J4.3, Q10.3; no longer D9.A, J2.3, Q4.3
- net N$67: now also D14.A, J4.2, Q29.3; no longer D10.A, J2.2, Q6.3
- net N$68: now also D13.A, J4.1, Q9.3; no longer D11.A, J2.1, Q8.3
- net N$69: now also Q28.3; no longer Q10.3
- net N$7: now also J30.5, U16.2; no longer J31.5, U22.2
- net N$70: now also D11.A, Q8.3; no longer D13.A, Q12.3
- net N$71: now also D10.A, Q27.3; no longer D14.A, Q14.3
- net N$72: now also D9.A, Q7.3; no longer D15.A, Q16.3
- net N$73: now also D8.A, J2.4, Q26.3; no longer D16.A, J4.4, Q18.3
- net N$74: now also D7.A, J2.3, Q6.3; no longer D17.A, J4.3, Q20.3
- net N$75: now also D13.C, R10.2; no longer D11.C, R41.2
- net N$76: now also J6.1, U2.1; no longer J10.1, U19.1
- net N$77: now also R9.2; no longer R43.2
- net N$78: now also D1.C, R14.2; no longer D27.C, R72.2
- net N$79: now also D2.C, R16.2; no longer D26.C, R71.2
- net N$8: now also J30.4, U16.1; no longer J31.4, U22.1
- net N$80: now also D3.C, R17.2; no longer D24.C, R69.2
- net N$81: now also D4.C, R1.2; no longer D25.C, R70.2
- net N$82: now also D14.C, R11.2; no longer D10.C, R39.2
- net N$83: now also D15.C, R12.2; no longer D9.C, R37.2
- net N$84: now also D16.C, R13.2; no longer D8.C, R35.2
- net N$85: now also D18.C, D20.A, D3.A, J1.3, Q23.3, Q3.3; no longer D20.C, D21.A, D24.A, J5.3, Q29.3, Q30.3
- net N$86: now also Q23.1, Q3.1, Q34.3, R38.1; no longer Q28.3, Q29.1, Q30.1, R61.1
- net N$87: now also Q34.1, U5.20; no longer Q28.1, U13.20
- net N$88: now also Q31.1, U5.19; no longer Q25.1, U13.19
- net N$89: now also D18.A, D20.C, R18.1; no longer D20.A, D21.C, R60.1
- net N$9: now also J30.3, U16.28; no longer J31.3, U22.28
- net N$90: now also Q35.1, U5.17; no longer Q21.1, U13.17
- net N$91: now also Q11.1, U5.18; no longer Q23.1, U13.18
- net N$92: now also D17.A, D19.C, R15.1; no longer D22.A, D23.C, R64.1
- net N$93: now also D6.A, J2.2, Q25.3; no longer D18.A, J4.2, Q22.3
- net N$94: now also D5.A, J2.1, Q5.3; no longer D19.A, J4.1, Q24.3
- net N$95: now also Q11.3, Q5.1, R27.1; no longer Q23.3, Q24.1, R56.1
- net N$96: now also Q25.1, Q35.3, R46.1; no longer Q21.3, Q22.1, R54.1
- net N$97: now also C4.1, R44.2, U6.3; no longer C15.1, R29.2, U10.3
- net N$98: now also D5.C, R2.2; no longer D19.C, R57.2
- net N$99: now also R54.1, R55.2, U6.6; no longer R31.2, R33.1, U10.6
- net RELAY0EN: now also Q20.1, U16.21; no longer Q43.1, U22.21
- net RELAY1EN: now also Q17.1, U16.22; no longer Q44.1, U22.22
- net RELAY2EN: now also Q19.1, U16.23; no longer Q45.1, U22.23
- net RELAY3EN: now also Q18.1, U16.24; no longer Q46.1, U22.24
- net RELAY4EN: now also R26.1, U16.25; no longer R88.1, U22.25
- net RELAY5EN: now also R25.1, U16.26; no longer R89.1, U22.26
- net RXEN: now also U3.4; no longer U7.4
- net S0: now also R41.1, S1.P$2; no longer R13.1, S0.P$2
- net S1: now also R42.1, S2.P$2; no longer R12.1, S1.P$2
- net SCL: now also J11.3, R40.1, U10.10, U16.12, U19.6, U20.SCL, U5.26, U7.4, U8.2; no longer J18.3, R94.1, U13.26, U2.6, U22.12, U3.2, U4.4, U6.SCL, U8.10
- net SDA: now also J11.4, R39.1, U10.9, U16.13, U19.5, U20.SDA, U5.27, U7.3, U8.1; no longer J18.4, R93.1, U13.27, U2.5, U22.13, U3.1, U4.3, U6.SDA, U8.9
- net SENSORS0: now also U18.11; no longer U21.11
- net SENSORS1: now also U18.10; no longer U21.10
- net SENSORS2: now also U18.9; no longer U21.9
- net STEPPER1DIROUT: now also J17.3, Q43.3; no longer J32.3, Q38.3
- net STEPPER1ENOUT: now also J17.4, Q44.3; no longer J32.4, Q37.3
- net STEPPERADIR: now also Q46.1, R84.2; no longer Q41.1, R77.2
- net STEPPERAEN: now also Q47.1, R85.2; no longer Q40.1, R76.2
- net STEPPERASTEP: now also Q45.1, R83.2; no longer Q42.1, R78.2
- net STEPPERBDIR: now also Q43.1, R81.2; no longer Q38.1, R74.2
- net STEPPERBEN: now also Q44.1, R82.2; no longer Q37.1, R73.2
- net STEPPERBSTEP: now also Q42.1, R80.2; no longer Q39.1, R75.2
- net TXEN: now also U3.3; no longer U7.3
- net UART0_RX: now also U3.2; no longer U7.2
- net UART0_TX: now also U3.5; no longer U7.5
- net VBATT: now also D31.C, J14.1, J15.1, J16.1, J16.2, J16.3, Q21.2, Q23.2, Q25.2, Q26.2, Q28.2, Q29.2, Q5.2, Q7.2, Q9.2, R19.2, R20.2, R21.2, R22.2, R23.2, R24.2, R27.2, R35.2, R37.2, R45.2, R47.2, R49.2, R51.2, U7.7, U9.IN+; no longer D4.C, J19.1, J19.2, J19.3, J8.1, J9.1, Q12.2, Q14.2, Q16.2, Q18.2, Q2.2, Q20.2, Q33.2, Q36.2, Q4.2, R34.2, R40.2, R42.2, R44.2, R52.2, R54.2, R56.2, R58.2, R61.2, R62.2, R65.2, R79.2, R91.2, U1.IN+, U4.7
- net VBATTISENSE: now also Q41.2, R51.1, U4.2, U4.3, U7.8; no longer Q47.2, R79.1, U4.8, U5.2, U5.3
