File: board/tex.brd (EAGLE design)
At the start: 200 x 100 mm, 270 parts, among them Q1 IRFZ44, Q10 FDD4141, Q11 2N7002, Q12 2N7002, Q13 2N7002, Q14 2N7002, Q15 2N7002, Q16 2N7002, Q17 2N7002, Q18 2N7002, Q19 2N7002, Q2 IRFZ44, Q20 2N7002, Q21 FDD4141, Q22 FDD4141, Q23 FDD4141, Q24 FDD4141, Q25 FDD4141, Q26 FDD4141, Q27 FDD4141, Q28 FDD4141, Q29 FDD4141, Q3 IRFZ44, Q30 FDD4141, Q31 2N7002, Q32 2N7002, Q33 2N7002, Q34 2N7002, Q35 2N7002, Q36 2N7002, Q37 2N7002, Q38 2N7002, Q39 2N7002, Q4 IRFZ44, Q40 2N7002, Q41 FDD4141, Q42 2N7002, Q43 2N7002, Q44 2N7002, Q45 2N7002, Q46 2N7002, Q47 2N7002, Q5 FDD4141, Q6 FDD4141, Q7 FDD4141, Q8 FDD4141, Q9 FDD4141, U10 ADS1x15, U11 DUALOPAMP, U12 OPTO-LTV817, U13 OPTO-LTV817, U14 OPTO-LTV817, U15 OPTO-LTV817, U16 MCP23017, U17 24LC32A, U18 IO-HC4051, U19 MCP7940N, U3 MAX13433E, U4 AZ23C5V1, U5 PCA9685, U6 DUALOPAMP, U7 INA219, U8 LM75, Y1 32.768KHz

Commit message: getting ready for first board run
Parts:
- R39, R40: value 120 -> 1k
- R73, R74: value 3.9k -> 1k
Changed lines of the file:
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@@
 <setting verticaltext="up"/>
 </settings>
-<grid distance="0.0196850394" unitdist="inch" unit="inch" style="lines" multiple="1" display="yes" altdistance="0.0025" altunitdist="inch" altunit="inch"/>
+<grid distance="1" unitdist="mm" unit="mm" style="lines" multiple="1" display="yes" altdistance="0.1" altunitdist="mm" altunit="mm"/>
 <layers>
 <layer number="1" name="Top" color="4" fill="1" visible="yes" active="yes"/>
@@
 <layer number="43" name="vRestrict" color="2" fill="10" visible="no" active="yes"/>
 <layer number="44" name="Drills" color="7" fill="1" visible="no" active="yes"/>
-<layer number="45" name="Holes" color="7" fill="1" visible="no" active="yes"/>
+<layer number="45" name="Holes" color="7" fill="1" visible="yes" active="yes"/>
 <layer number="46" name="Milling" color="3" fill="1" visible="no" active="yes"/>
 <layer number="47" name="Measures" color="7" fill="1" visible="no" active="yes"/>
@@
 <attribute name="VALUE" x="158.542" y="83.71" size="1.016" layer="27" ratio="21" rot="R180"/>
 </element>
-<element name="R73" library="holla" package="R0603" value="3.9k" x="155" y="73" smashed="yes">
+<element name="R73" library="holla" package="R0603" value="1k" x="155" y="73" smashed="yes">
 <attribute name="NAME" x="155.05" y="73.666" size="1.016" layer="25" ratio="21" align="bottom-center"/>
 <attribute name="VALUE" x="155" y="71.984" size="1.016" layer="27" ratio="21" align="top-center"/>
 <attribute name="DESC" value="5%" x="155" y="73" size="1.778" layer="27" display="off"/>
 </element>
-<element name="R74" library="holla" package="R0603" value="3.9k" x="151.658" y="73.674" smashed="yes" rot="R270">
+<element name="R74" library="holla" package="R0603" value="1k" x="151.658" y="73.674" smashed="yes" rot="R270">
 <attribute name="NAME" x="152.374" y="73.674" size="1.016" layer="25" ratio="21" rot="R270" align="bottom-center"/>
 <attribute name="VALUE" x="150.642" y="73.674" size="1.016" layer="27" ratio="21" rot="R270" align="top-center"/>
@@
 <attribute name="VALUE" x="187.841" y="55.06" size="1.27" layer="27" rot="R270"/>
 </element>
-<element name="R39" library="holla" package="R0603" value="120" x="152.968" y="44" smashed="yes" rot="R270">
+<element name="R39" library="holla" package="R0603" value="1k" x="152.968" y="44" smashed="yes" rot="R270">
 <attribute name="NAME" x="151.134" y="44.05" size="1.016" layer="25" ratio="21" rot="R270" align="bottom-center"/>
 <attribute name="VALUE" x="151.952" y="44" size="1.016" layer="27" ratio="21" rot="R270" align="top-center"/>
 <attribute name="DESC" value="5%" x="152.968" y="44" size="1.778" layer="27" rot="R270" display="off"/>
 </element>
-<element name="R40" library="holla" package="R0603" value="120" x="155.294" y="44" smashed="yes" rot="R270">
+<element name="R40" library="holla" package="R0603" value="1k" x="155.294" y="44" smashed="yes" rot="R270">
 <attribute name="NAME" x="156.31" y="44" size="1.016" layer="25" ratio="21" rot="R270" align="bottom-center"/>
 <attribute name="VALUE" x="154.278" y="44" size="1.016" layer="27" ratio="21" rot="R270" align="top-center"/>

Commit message: initial add for blink
Parts:
- added U22: DUALOPAMP, holla:SO08
- B1: value (none) -> CR2032
- D35, D36: device holla:SOD-323 -> holla:SOD-523
- Q1, Q2, Q3, Q4: value IRFZ44 -> FET-NCH
- Q10, Q21, Q22, Q23, Q24, Q25, Q26, Q27, Q28, Q29, Q30, Q41, Q5, Q6, Q7, Q8, Q9: value FDD4141 -> FET-PCH
- Q11, Q12, Q13, Q14, Q15, Q16, Q17, Q18, Q19, Q20, Q31, Q32, Q33, Q34, Q35, Q36, Q37, Q38, Q39, Q40, Q42, Q43, Q44, Q45, Q46, Q47: value 2N7002 -> FET-NCH
- S1, S2: value (none) -> UI
- U12, U13, U14, U15: value OPTO-LTV817 -> OPTO
Connections:
- new net V+: U22.8
- new net V-: U22.4

Commit message: added todo items
Parts:
- F1: value 20A -> 10A
- R33, R34: value 1 -> 0.1
- R51: value 10 -> 0.1
Changed lines of the file:
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@@
 <attribute name="VALUE" x="109.35" y="85.94" size="1.27" layer="27"/>
 </element>
-<element name="F1" library="holla" package="3557-2" value="20A" x="9" y="65" smashed="yes" rot="R270">
+<element name="F1" library="holla" package="3557-2" value="10A" x="9" y="65" smashed="yes" rot="R270">
 <attribute name="NAME" x="12.81" y="73.89" size="1.016" layer="25" ratio="21" rot="R270"/>
 <attribute name="VALUE" x="3.92" y="73.89" size="1.016" layer="27" ratio="21" rot="R270"/>
@@
 <attribute name="VALUE" x="0.92" y="22.54" size="1.27" layer="27" rot="R270"/>
 </element>
-<element name="R33" library="holla" package="R1210" value="1" x="11.246" y="40" smashed="yes" rot="R90">
+<element name="R33" library="holla" package="R1210" value="0.1" x="11.246" y="40" smashed="yes" rot="R90">
 <attribute name="NAME" x="11.45" y="37.518" size="1.016" layer="25" ratio="21" rot="R180" align="bottom-center"/>
 <attribute name="VALUE" x="13.024" y="40" size="1.016" layer="27" ratio="21" rot="R90" align="top-center"/>
@@
 <attribute name="VALUE" x="19.92" y="22.54" size="1.27" layer="27" rot="R270"/>
 </element>
-<element name="R34" library="holla" package="R1210" value="1" x="30.5" y="40" smashed="yes" rot="R90">
+<element name="R34" library="holla" package="R1210" value="0.1" x="30.5" y="40" smashed="yes" rot="R90">
 <attribute name="NAME" x="30.65" y="37.472" size="1.016" layer="25" ratio="21" rot="R180" align="bottom-center"/>
 <attribute name="VALUE" x="32.278" y="40" size="1.016" layer="27" ratio="21" rot="R90" align="top-center"/>
@@
 <attribute name="VALUE" x="25.135" y="11.405" size="1.27" layer="27" rot="R180"/>
 </element>
-<element name="R51" library="holla" package="R1210" value="10" x="24.13" y="49.022" smashed="yes" rot="R270">
+<element name="R51" library="holla" package="R1210" value="0.1" x="24.13" y="49.022" smashed="yes" rot="R270">
 <attribute name="NAME" x="27.428" y="49.658" size="1.016" layer="25" ratio="21" align="bottom-center"/>
 <attribute name="VALUE" x="22.352" y="49.022" size="1.016" layer="27" ratio="21" rot="R270" align="top-center"/>
