File: board/tex.brd (EAGLE design)
At the start: 200 x 100 mm, 271 parts, among them Q1 FET-NCH, Q10 FET-PCH, Q11 FET-NCH, Q12 FET-NCH, Q13 FET-NCH, Q14 FET-NCH, Q15 FET-NCH, Q16 FET-NCH, Q17 FET-NCH, Q18 FET-NCH, Q19 FET-NCH, Q2 FET-NCH, Q20 FET-NCH, Q21 FET-PCH, Q22 FET-PCH, Q23 FET-PCH, Q24 FET-PCH, Q25 FET-PCH, Q26 FET-PCH, Q27 FET-PCH, Q28 FET-PCH, Q29 FET-PCH, Q3 FET-NCH, Q30 FET-PCH, Q31 FET-NCH, Q32 FET-NCH, Q33 FET-NCH, Q34 FET-NCH, Q35 FET-NCH, Q36 FET-NCH, Q37 FET-NCH, Q38 FET-NCH, Q39 FET-NCH, Q4 FET-NCH, Q40 FET-NCH, Q41 FET-PCH, Q42 FET-NCH, Q43 FET-NCH, Q44 FET-NCH, Q45 FET-NCH, Q46 FET-NCH, Q47 FET-NCH, Q5 FET-PCH, Q6 FET-PCH, Q7 FET-PCH, Q8 FET-PCH, Q9 FET-PCH, U10 ADS1x15, U11 DUALOPAMP, U12 OPTO, U13 OPTO, U14 OPTO, U15 OPTO, U16 MCP23017, U17 24LC32A, U18 IO-HC4051, U19 MCP7940N, U22 DUALOPAMP, U3 MAX13433E, U4 AZ23C5V1, U5 PCA9685, U6 DUALOPAMP, U7 INA219, U8 LM75, Y1 32.768KHz

Commit message: more notes
Parts:
- C13, C14: value 12p -> 6p
Changed lines of the file:
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@@
 <attribute name="DESC" value="5%" x="190" y="80.5" size="1.778" layer="27" rot="R180" display="off"/>
 </element>
-<element name="C13" library="holla" package="C0603" value="12p" x="189" y="75.5" smashed="yes" rot="R90">
+<element name="C13" library="holla" package="C0603" value="6p" x="189" y="75.5" smashed="yes" rot="R90">
 <attribute name="NAME" x="189.538" y="72.55" size="1.016" layer="25" ratio="21" rot="R90" align="bottom-center"/>
 <attribute name="VALUE" x="189.762" y="75.5" size="1.016" layer="27" ratio="21" rot="R90" align="top-center"/>
 <attribute name="DESC" value="16V Y5V -20%,+80%" x="189" y="75.5" size="1.778" layer="27" rot="R90" display="off"/>
 </element>
-<element name="C14" library="holla" package="C0603" value="12p" x="197" y="75.5" smashed="yes" rot="R90">
+<element name="C14" library="holla" package="C0603" value="6p" x="197" y="75.5" smashed="yes" rot="R90">
 <attribute name="NAME" x="197.688" y="72.65" size="1.016" layer="25" ratio="21" rot="R90" align="bottom-center"/>
 <attribute name="VALUE" x="197.762" y="75.5" size="1.016" layer="27" ratio="21" rot="R90" align="top-center"/>
