File: board/tex.sch (EAGLE design)
At the start: 179 parts, among them U2 RTC-DS1337S, Y1 32.768KHz

Commit message: continuing work on sch
Parts:
- removed JBATT, JGND, JP5, JP6, JP7, JP8: (no value), holla:M051.27MM
- added D24, D25, D26, D27, D32, D33, D34, D35: (no value), holla:LED-0603
- added D28, D29, D30, D31: (no value), holla:DIODE-0603
- added J1: (no value), holla:M02-6.35MM
- added J11, J12, J13, J14: (no value), holla:M03-1984620
- added J2, J3, J4, J5, J6, J7, J8, J9: (no value), holla:M04-1984633
- added JP9: DNP, holla:JUMPER-PAD-2-NO
- added K1, K2, K3, K4: HLS8L-DC5V-S-C, holla:RELAY-HLS8L-DC5V-S-C(5P-19X15MM)
- added Q37, Q38, Q39, Q40, Q41, Q42, Q43, Q44, Q45, Q46: (no value), holla:FET-NCHANNEL-SOT23
- added R66: 1k, holla:R-US_R0603
- added R67, R68: 3.9k, holla:R-US_R0603
- added R69, R70, R71, R72, R73, R74, R75, R76, R77, R78, R80, R81, R82, R83, R84, R85, R86, R87: (no value), holla:R-US_R0603
- added R79: (no value), holla:R-US_R1210
- added U14: 24LC32A, holla:MEMORY-EEPROM-SO08
- added U15, U16, U17, U18: OPTO-LTV817, holla:OPTO-LTV817
Connections:
- removed net N$76: D16.A, R51.1
- new net DCMOTOR1ENCA: U15.4
- new net DCMOTOR1ENCB: U16.4
- new net DCMOTOR2ENCA: U17.4
- new net DCMOTOR2ENCB: U18.4
- new net GND4: D31.A, D35.C, K4.V-, Q46.D
- new net ID_SC: PCB1.ID_SC*, R67.1, U14.SCL
- new net ID_SD: PCB1.ID_SD*, R68.1, U14.SDA
- new net N$102: PCB1.5V@2
- new net N$103: PCB1.5V@4
- new net N$104: JP9.2, R66.1, U14.WP
- new net N$106: PCB1.GND@6
- new net N$108: PCB1.GPIO14
- new net N$109: PCB1.GPIO15
- new net N$110: PCB1.GPIO18
- new net N$111: PCB1.GND@14
- new net N$112: PCB1.GPIO23
- new net N$113: PCB1.GPIO24
- new net N$114: PCB1.GND@20
- new net N$115: PCB1.GPIO25
- new net N$116: PCB1.GPIO8
- new net N$117: PCB1.GPIO7
- new net N$118: PCB1.GND@30
- new net N$119: PCB1.GPIO12
- new net N$120: PCB1.GND@34
- new net N$121: PCB1.GPIO16
- new net N$122: PCB1.GPIO20
- new net N$123: PCB1.GPIO21
- new net N$124: PCB1.GND@39
- new net N$125: PCB1.GPIO26
- new net N$126: PCB1.GPIO19
- new net N$127: PCB1.GPIO13
- new net N$128: PCB1.GPIO6
- new net N$129: PCB1.GPIO5
- new net N$130: PCB1.GND@25
- new net N$131: PCB1.GPIO11
- new net N$132: PCB1.GPIO9
- new net N$133: PCB1.GPIO10
- new net N$134: PCB1.3V3@17
- new net N$135: PCB1.GPIO22
- new net N$136: PCB1.GPIO27
- new net N$137: PCB1.GPIO17
- new net N$138: PCB1.GND@9
- new net N$139: D17.C, R53.2
- new net N$140: D16.C, R51.2
- new net N$141: D15.C, R49.2
- new net N$142: D14.C, R47.2
- new net N$143: J14.2, K1.COM
- new net N$144: J14.1, K1.NO
- new net N$145: J14.3, K1.NC
- new net N$146: D13.C, R45.2
- new net N$147: D33.A, R85.1
- new net N$148: R80.1, U15.1
- new net N$149: J8.3, R81.2
- new net N$150: J8.2, R80.2
- new net N$151: J6.4, Q39.D
- new net N$152: J7.2, Q40.D
- new net N$153: J7.3, Q41.D
- new net N$154: J7.4, Q42.D
- new net N$155: R81.1, U16.1
- new net N$156: J9.2, R82.2
- new net N$157: J9.3, R83.2
- new net N$158: R82.1, U17.1
- new net N$159: D30.A, D34.C, K3.V-, Q45.D
- new net N$160: D28.C, D29.C, D30.C, D31.C, K1.V+, K2.V+, K3.V+, K4.V+, R85.2, R86.2, R87.2
- new net N$161: D29.A, D33.C, K2.V-, Q44.D
- new net N$162: R83.1, U18.1
- new net N$163: J11.2, K2.COM
- new net N$164: J11.1, K2.NO
- new net N$165: J11.3, K2.NC
- new net N$166: J12.2, K3.COM
- new net N$167: J12.1, K3.NO
- new net N$168: J12.3, K3.NC
- new net N$169: J13.1, K4.NO
- new net N$170: J13.2, K4.COM
- new net N$171: J13.3, K4.NC
- new net N$172: R84.2
- new net N$173: D32.A, R84.1
- new net N$174: D34.A, R86.1
- new net N$175: D35.A, R87.1
- new net N$176: D28.A, D32.C, K1.V-, Q43.D
- new net RELAY1EN: Q43.G
- new net RELAY2EN: Q44.G
- new net RELAY3EN: Q45.G
- new net RELAY4EN: Q46.G
- new net STEPPER1DIR: Q38.G, R74.2
- new net STEPPER1DIROUT: J6.3, Q38.D
- new net STEPPER1EN: Q37.G, R73.2
- new net STEPPER1ENOUT: J6.2, Q37.D
- new net STEPPER1STEP: Q39.G, R75.2
- new net STEPPER2DIR: Q41.G, R77.2
- new net STEPPER2EN: Q40.G, R76.2
- new net STEPPER2STEP: Q42.G, R78.2
- new net VBATTISENSE: F1.P$2, R79.1
- net +5V: now also J6.1, J7.1
- net GND: now also J1.1, J8.4, J9.4, JP9.1, Q37.S, Q38.S, Q39.S, Q40.S, Q41.S, Q42.S, Q43.S, Q44.S, Q45.S, Q46.S, R35.1, R37.1, R39.1, R41.1, R43.1, R45.1, R47.1, R49.1, R51.1, R53.1, R55.1, R57.1, R69.1, R70.1, R71.1, R72.1, R73.1, R74.1, R75.1, R76.1, R77.1, R78.1, U14.A0, U14.A1, U14.A2, U14.GND, U15.2, U15.3, U16.2, U16.3, U17.2, U17.3, U18.2, U18.3; no longer D10.C, D11.C, D12.C, D13.C, D14.C, D15.C, D16.C, D17.C, D18.C, D19.C, D8.C, D9.C, JGND.1, JGND.2, JGND.3, JGND.4, JGND.5, JP5.1, JP6.1, JP7.1, JP8.1
- net N$100: now also D18.C, R55.2; no longer D19.A, R57.1
- net N$101: now also J1.2; no longer JBATT.1, JBATT.2, JBATT.3, JBATT.4, JBATT.5
- net N$57: now also D26.A, J5.2; no longer JP8.3
- net N$59: now also D27.A, J5.1; no longer JP8.2
- net N$61: no longer Q34.G
- net N$63: now also D25.A, J5.4; no longer JP8.5
- net N$65: now also D8.A, J2.4; no longer JP5.5, R35.2
- net N$66: now also D9.A, J2.3; no longer JP5.4, R37.2
- net N$67: now also D10.A, J2.2; no longer JP5.3, R39.2
- net N$68: now also D11.A, J2.1; no longer R41.2
- net N$69: now also D12.A, J3.4; no longer JP6.5, R43.2
- net N$70: now also D13.A, J3.3; no longer JP6.4, R45.2
- net N$71: now also D14.A, J3.2; no longer JP6.3, R47.2
- net N$72: now also D15.A, J3.1; no longer JP6.2, R49.2
- net N$73: now also D16.A, J4.4; no longer JP7.5, R51.2
- net N$74: now also D17.A, J4.3; no longer JP7.4, R53.2
- net N$75: now also D11.C, R41.2; no longer D17.A, R53.1
- net N$77: now also D12.C, R43.2; no longer D15.A, R49.1
- net N$78: now also D27.C, R72.2; no longer D14.A, R47.1
- net N$79: now also D26.C, R71.2; no longer D13.A, R45.1
- net N$80: now also D24.C, R69.2; no longer D12.A, R43.1
- net N$81: now also D25.C, R70.2; no longer D11.A, R41.1
- net N$82: now also D10.C, R39.2; no longer D10.A, R39.1
- net N$83: now also D9.C, R37.2; no longer D9.A, R37.1
- net N$84: now also D8.C, R35.2; no longer D8.A, R35.1
- net N$85: now also D24.A, J5.3; no longer JP8.4
- net N$93: now also D18.A, J4.2; no longer JP7.3, R55.2
- net N$94: now also D19.A, J4.1; no longer JP7.2, R57.2
- net N$98: now also D19.C, R57.2; no longer D18.A, R55.1
- net VBATT: now also J8.1, J9.1, R79.2; no longer F1.P$2
- net VCC: now also R66.2, R67.2, R68.2, U14.VCC
Other:
- note added: "add current sense at the fuse level add I2C oled display add clamp to incoming voltage, motor spikes"
- note added: "put INA219 here add +5V out connector for stepper driver"
- note removed: "WiFi"
- note removed: "add motor encoder inputs"
- note removed: "uSD"
- moved on the sheet: D10, D11, D12, D13, D14, D15, D16, D17, D18, D19, D20, D21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

Commit message: mostly layout changes
Parts:
- removed $5_223_$_2016-03-04_22-58-43, $5_224_$_2016-03-04_22-58-43, TP1, TP2, TP3, TP4: (no value), holla:TESTPOINTTHRU
- removed C10, C11, C12, C13, C14, C18, C19, C20, C21, C4, C5, C6, C7, C8, C9: .1u, holla:C-USC0603
- removed C23: (no value), holla:C-USC0603
- removed D4, D5, D6, D7: (no value), holla:PROTECTION-TVS0603
- removed J6: (no value), holla:M04-1984633
- removed JP1, JP2, JP3, JP4: DNP, holla:JUMPER-PAD-2-NO
- removed R11, R16, R17, R18, R19, R20, R21, R22, R23, R6, R7, R8, R9: 1k, holla:R-US_R0603
- removed R12, R13, R14, R15: 10k, holla:R-US_R0603
- removed R24, R25, R26, R27: 100, holla:R-US_R0603
- removed U11, U12, U9: (no value), holla:ADC-ADS1015-MSOP10
- removed U6, U7: (no value), holla:AMP-OPAMP-DUAL-SO08
- added C24, C25, C26, C27, C28, C29, C30, C31, C32, C33, C34, C35, C36, C37, C38: (no value), holla:C-USC0603
- added D36, D37: (no value), holla:LED-0603
- added J10, J15, J23, J24, J25, J26, J27, J28: (no value), holla:M02-PLUGIN-SCREW
- added J16: OLED DISPLAY, holla:M04-0.1
- added J17, J18, J19, J20, J21, J22, J31: (no value), holla:M06-PLUGIN-SCREW
- added J29, J30: (no value), holla:M03-PLUGIN-SCREW
- added J32: (no value), holla:M05-PLUGIN-SCREW
- added Q47: FDD4141, brightleaf:FDD4141TO252
- added R88, R89, R92, R93, R94, R95: (no value), holla:R-US_R0603
- added R90: DNP, holla:R-US_R0603
- added R91: 0, holla:R-US_R0603
- added U19, U20: RELAY-S108T02PTH, holla:RELAY-S108T02PTH
- added U21: IO-HC4051, holla:IO-HC4051
- added U22: (no value), holla:IO-MCP23017SO
- C3: value .1u -> (none)
- J11, J12, J13, J14: device holla:M03-1984620 -> holla:M03-PLUGIN-SCREW
- J2, J3, J4, J5, J8, J9: device holla:M04-1984633 -> holla:M04-PLUGIN-SCREW
- J7: device holla:M04-1984633 -> holla:M05-PLUGIN-SCREW
- R10: value 1k -> 47k; device holla:R-US_R0603 -> rcl:R-US_R0402
- R4, R5: value 1k -> (none)
- R59, R63: device holla:R-US_R0603 -> holla:R-US_R1210
- U4: device holla:AMP-OPAMP-DUAL-SO08 -> holla:ADC-INA219-SOIC8
- U5: value (none) -> AZ23C5V1; device holla:AMP-OPAMP-DUAL-SO08 -> brightleaf:AZ23CXXX
Connections:
- net N$108 renamed UART0_TX
- net N$109 renamed UART0_RX
- removed net ADC0_0: U8.AIN0
- removed net ADC1_0: U9.AIN0
- removed net ADC1_1: U9.AIN1
- removed net ADC1_2: U9.AIN2
- removed net ADC1_3: U9.AIN3
- removed net ADC2_0: D6.1, R26.2, TP1.P$1, U11.AIN0
- removed net ADC2_1: D7.1, R27.2, TP2.P$1, U11.AIN1
- removed net ADC2_2: D4.1, R24.2, TP3.P$1, U11.AIN2
- removed net ADC2_3: D5.1, R25.2, TP4.P$1, U11.AIN3
- removed net ADC3_0: R30.2, U10A.OUT, U12.AIN0
- removed net ADC3_1: R33.2, U10B.OUT, U12.AIN1
- removed net ADC3_2: U12.AIN2
- removed net ADC3_3: U12.AIN3
- removed net N$10: R10.2, R11.2, R15.1, U7A.-IN
- removed net N$11: U7A.+IN
- removed net N$12: JP4.2, R10.1
- removed net N$13: C11.1, R20.2, U4B.-IN
- removed net N$14: JP3.2, R8.1
- removed net N$15: C7.1, R24.1, U4B.+IN, U4B.OUT
- removed net N$16: C7.2, R16.2, R20.1
- removed net N$17: R12.2, R16.1, U4A.OUT
- removed net N$18: C9.1, R26.1, U6B.+IN, U6B.OUT
- removed net N$19: R12.1, R4.2, R5.2, U4A.-IN
- removed net N$20: U4A.+IN
- removed net N$21: JP1.2, R4.1
- removed net N$22: C12.1, R21.2, U5B.-IN
- removed net N$23: C8.1, R25.1, U5B.+IN, U5B.OUT
- removed net N$24: C8.2, R17.2, R21.1
- removed net N$25: R13.2, R17.1, U5A.OUT
- removed net N$26: R13.1, R6.2, R7.2, U5A.-IN
- removed net N$27: U5A.+IN
- removed net N$28: JP2.2, R6.1
- removed net N$38: R14.2, R18.1, U6A.OUT
- removed net N$39: R14.1, R8.2, R9.2, U6A.-IN
- removed net N$55: U6A.+IN
- removed net SUPPLY: C1.1, U2.VCC
- removed net VCC: C18.1, C19.1, C2.1, C20.1, C21.1, C22.1, C23.1, R66.2, R67.2, R68.2, U11.VCC, U12.VCC, U13.A0, U13.A2, U13.A4, U13.VCC, U14.VCC, U3.VCC, U8.VCC, U9.ADDR, U9.VCC
- new net +3V3: J22.1, J22.2, J22.3, J22.4, J22.5, J22.6, PCB1.3V3@1, R66.2, R67.2, R68.2, U14.VCC
- new net C_24IN: F1.P$2, Q47.D
- new net INPUTINTERRUPT: U22.INTB
- new net N$108: C26.1, J17.3, U22.GPB4
- new net N$109: C27.1, J17.4, U22.GPB5
- new net N$177: J10.2, U19.T2
- new net N$178: J15.1, U20.T1
- new net N$179: J15.2, U20.T2
- new net N$180: D36.C, R88.2
- new net N$181: D37.C, R89.2
- new net N$182: D36.A, U19.-
- new net N$183: D37.A, U20.-
- new net N$184: C34.1, J26.2, U21.Y4
- new net N$185: C35.1, J25.2, U21.Y5
- new net N$186: C36.1, J24.2, U21.Y6
- new net N$187: C37.1, J23.2, U21.Y7
- new net N$76: J10.1, U19.T1
- new net RELAY0EN: Q43.G, U22.GPA0
- new net RELAY5EN: R89.1, U22.GPA5
- new net SENSORS0: U21.S0
- new net SENSORS1: U21.S1
- new net SENSORS2: U21.S2
- net +5V: now also C1.1, C2.1, C22.1, C3.1, C38.1, J16.2, J20.1, J20.2, J20.3, J20.4, J20.5, J20.6, J29.3, J30.3, J31.6, J32.5, J7.5, PCB1.5V@2, PCB1.5V@4, R90.2, R92.2, R93.2, R94.2, R95.2, U13.A5, U13.VCC, U19.+, U2.VCC, U20.+, U21.VCC, U22.!RESET, U22.VDD, U3.A2, U3.VCC, U4.VS, U8.VCC; no longer J6.1, J7.1
- net ADC0_1: now also R30.2, U10A.OUT
- net ADC0_2: now also R33.2, U10B.OUT
- net AGND: no longer C11.2, C12.2, C13.2, C14.2, C15.2, C16.2, C17.2, C3.2, C4.2, C5.2, C6.2, D4.2, D5.2, D6.2, D7.2, JP1.1, JP2.1, JP3.1, JP4.1, R11.1, R5.1, R7.1, R9.1, U10A.V-, U4A.V-, U5A.V-, U6A.V-, U7A.V-
- net AVCC: no longer C3.1, C4.1, C5.1, C6.1, U4A.V+, U5A.V+, U6A.V+, U7A.V+
- net GND: now also C15.2, C16.2, C17.2, C24.2, C25.2, C26.2, C27.2, C28.2, C29.2, C3.2, C30.2, C31.2, C32.2, C33.2, C34.2, C35.2, C36.2, C37.2, C38.2, J16.1, J18.1, J18.2, J18.3, J18.4, J18.5, J18.6, J21.1, J21.2, J21.3, J21.4, J21.5, J21.6, J23.1, J24.1, J25.1, J26.1, J27.1, J28.1, J29.1, J30.1, J31.1, J32.1, J7.1, PCB1.GND@14, PCB1.GND@20, PCB1.GND@25, PCB1.GND@30, PCB1.GND@34, PCB1.GND@39, PCB1.GND@6, PCB1.GND@9, R10.1, R5.1, U10A.V-, U13.A0, U13.A2, U13.A4, U21.!E, U21.GND, U21.VEE, U22.A0, U22.A1, U22.A2, U22.VSS, U4.A0, U4.A1, U4.GND; no longer C18.2, C19.2, C20.2, C21.2, C23.2, U11.GND, U12.GND, U13.A5, U3.A2, U9.GND
- net N$102: now also C24.1, J17.1, U22.GPB2; no longer PCB1.5V@2
- net N$103: now also C25.1, J17.2, U22.GPB3; no longer PCB1.5V@4
- net N$106: now also PCB1.GPIO4; no longer PCB1.GND@6
- net N$111: now also C28.1, J17.5, U22.GPB6; no longer PCB1.GND@14
- net N$114: now also C29.1, J17.6, U22.GPB7; no longer PCB1.GND@20
- net N$118: now also U21.Z, U8.AIN0; no longer PCB1.GND@30
- net N$120: now also C30.1, J30.2, R92.1, U21.Y0; no longer PCB1.GND@34
- net N$124: now also C31.1, J29.2, R93.1, U21.Y1; no longer PCB1.GND@39
- net N$130: now also C32.1, R4.1, R5.2, R94.1, U21.Y2; no longer PCB1.GND@25
- net N$138: now also C33.1, J27.2, R95.1, U21.Y3; no longer PCB1.GND@9
- net N$151: now also J32.2; no longer J6.4
- net N$152: now also J7.4; no longer J7.2
- net N$154: now also J7.2; no longer J7.4
- net N$172: now also R90.1, R91.1
- net N$2: now also J28.2, R4.2; no longer C14.1, R23.2, U7B.-IN
- net N$4: now also Q47.G, R10.2, U5.A; no longer C10.1, R27.1, U7B.+IN, U7B.OUT
- net N$6: now also J31.5, U22.GPA6; no longer C10.2, R19.2, R23.1
- net N$7: now also J31.4, U22.GPA7; no longer C9.2, R18.2, R22.1
- net N$8: now also J31.3, U22.GPB0; no longer C13.1, R22.2, U6B.-IN
- net N$9: now also J31.2, U22.GPB1; no longer R15.2, R19.1, U7A.OUT
- net RELAY1EN: now also Q44.G, U22.GPA1; no longer Q43.G
- net RELAY2EN: now also Q45.G, U22.GPA2; no longer Q44.G
- net RELAY3EN: now also Q46.G, U22.GPA3; no longer Q45.G
- net RELAY4EN: now also R88.1, U22.GPA4; no longer Q46.G
- net SCL: now also J16.3, PCB1.GPIO3, U22.SCL, U4.SCL; no longer $5_224_$_2016-03-04_22-58-43.P$1, U11.SCL, U12.ADDR, U12.SCL, U9.SCL
- net SDA: now also J16.4, PCB1.GPIO2, U22.SDA, U4.SDA; no longer $5_223_$_2016-03-04_22-58-43.P$1, U11.ADDR, U11.SDA, U12.SDA, U9.SDA
- net STEPPER1DIROUT: now also J32.3; no longer J6.3
- net STEPPER1ENOUT: now also J32.4; no longer J6.2
- net VBATT: now also J19.1, J19.2, J19.3, J19.4, J19.5, J19.6, R91.2, U4.IN-
- net VBATTISENSE: now also Q47.S, U4.IN+, U5.C1, U5.C2; no longer F1.P$2
Other:
- note added: "AC Current ~1VAC"
- note added: "AC Voltage ~9VAC"
- note added: "AGND not implemented, not high-performance design I2C Address Table 010 0000 I/O MCP23107 100 0000 VBATT Current Sense INA219 100 1000 ADC ADS1015 100 1100 TEMP LM75 110 0000 LED PCA9685 110 1000 RTC DS1337 111 1000 Display SSD1306 Banggood"
- note added: "MUX"
- note added: "NTC 10K Thermistors"
- note added: "Reverse Protection"
- note added: "Sensors"
- note added: "Spare"
- note added: "Water Pressure"
- note added: "addr 010 0000"
- note added: "addr 100 0000"
- note added: "addr 100 1000"
- note added: "addr 100 1100"
- note added: "addr 110 0000"
- note added: "addr 110 1000"
- note added: "addr 111 1000"
- note added: "external user switch inputs"
- note added: "http://hackaday.com/2011/12/06/reverse-voltage-protection-with-a-p-fet/"
- note added: "put MAX13433E here"
- note added: "put down analog gnds add +5V out connector for stepper driver"
- note removed: "1.6kHz Low Pass"
- note removed: "ADC1"
- note removed: "ADC2"
- note removed: "ADC3"
- note removed: "I2C address = 1010 101x."
- note removed: "NEED TO CHECK I2C ADDR CONFLICTS"
- note removed: "Photocell"
- note removed: "clamp"
- note removed: "put INA219 here add +5V out connector for stepper driver"

Commit message: parts placed
Parts:
- removed J18, J20, J22: (no value), holla:M06-PLUGIN-SCREW
- added C4, C5: .1u, holla:C-USC0603
- added D4: (no value), holla:DIODE-SMA
- added J6: (no value), holla:M05-PLUGIN-SCREW
- added R11: 120, holla:R-US_R0603
- added R12, R13, R14, R15, R6, R7, R8, R9: (no value), holla:R-US_R0603
- added S1, S2, S3, S4: (no value), holla:SWITCH-PUSHBUTTON-6MMX3.5MM
- added U6: (no value), holla:DISP-I2C-4PIN
- added U7: (no value), holla:COMM-MAX13433E
- J16: value OLED DISPLAY -> (none); device holla:M04-0.1 -> holla:M02-0.1
Connections:
- new net N$10: U7.DI
- new net N$11: U7.RO
- new net N$12: U7.!RE
- new net N$13: J6.2, R11.2, U7.A
- new net N$14: J6.3, R11.1, U7.B
- new net N$15: J6.4, U7.Y
- new net N$16: J6.5, U7.Z
- new net N$17: J16.2, J6.1
- new net N$19: U7.DE
- new net N$21: R15.1, S1.2
- new net N$22: R14.1, S2.2
- new net N$23: R13.1, S3.2
- new net N$24: R12.1, S4.2
- net +3V3: now also C5.1, R12.2, R13.2, R14.2, R15.2, U7.VL; no longer J22.1, J22.2, J22.3, J22.4, J22.5, J22.6
- net +5V: now also C4.1, J19.4, J19.5, J19.6, R6.2, R7.2, R8.2, R9.2, U6.VCC, U7.VCC; no longer J16.2, J20.1, J20.2, J20.3, J20.4, J20.5, J20.6
- net GND: now also C4.2, C5.2, D4.A, S1.1, S2.1, S3.1, S4.1, U6.GND, U7.GND6, U7.GND8; no longer J18.1, J18.2, J18.3, J18.4, J18.5, J18.6
- net N$184: now also R6.1
- net N$185: now also R7.1
- net N$186: now also R8.1
- net N$187: now also R9.1
- net N$6: now also J31.2; no longer J31.5
- net N$7: now also J31.5, U22.GPB1; no longer J31.4, U22.GPA7
- net N$8: now also J31.4; no longer J31.3
- net N$9: now also J31.3, U22.GPA7; no longer J31.2, U22.GPB1
- net SCL: now also U6.SCL; no longer J16.3
- net SDA: now also U6.SDA; no longer J16.4
- net VBATT: now also D4.C; no longer J19.4, J19.5, J19.6
