File: board/tex.sch (EAGLE design)
At the start: 270 parts, among them Q1 IRFZ44, Q10 FDD4141, Q11 2N7002, Q12 2N7002, Q13 2N7002, Q14 2N7002, Q15 2N7002, Q16 2N7002, Q17 2N7002, Q18 2N7002, Q19 2N7002, Q2 IRFZ44, Q20 2N7002, Q21 FDD4141, Q22 FDD4141, Q23 FDD4141, Q24 FDD4141, Q25 FDD4141, Q26 FDD4141, Q27 FDD4141, Q28 FDD4141, Q29 FDD4141, Q3 IRFZ44, Q30 FDD4141, Q31 2N7002, Q32 2N7002, Q33 2N7002, Q34 2N7002, Q35 2N7002, Q36 2N7002, Q37 2N7002, Q38 2N7002, Q39 2N7002, Q4 IRFZ44, Q40 2N7002, Q41 FDD4141, Q42 2N7002, Q43 2N7002, Q44 2N7002, Q45 2N7002, Q46 2N7002, Q47 2N7002, Q5 FDD4141, Q6 FDD4141, Q7 FDD4141, Q8 FDD4141, Q9 FDD4141, U10 ADS1x15, U11 DUALOPAMP, U12 OPTO-LTV817, U13 OPTO-LTV817, U14 OPTO-LTV817, U15 OPTO-LTV817, U16 MCP23017, U17 24LC32A, U18 IO-HC4051, U19 MCP7940N, U3 MAX13433E, U4 AZ23C5V1, U5 PCA9685, U6 DUALOPAMP, U7 INA219, U8 LM75, Y1 32.768KHz

Commit message: getting ready for first board run
Parts:
- R39, R40: value 120 -> 1k
- R73, R74: value 3.9k -> 1k
Changed lines of the file:
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@@
 <grid distance="0.1" unitdist="inch" unit="inch" style="lines" multiple="1" display="yes" altdistance="0.01" altunitdist="inch" altunit="inch"/>
 <layers>
-<layer number="1" name="Top" color="4" fill="1" visible="no" active="no"/>
-<layer number="2" name="Route2" color="1" fill="3" visible="no" active="no"/>
-<layer number="3" name="Route3" color="4" fill="3" visible="no" active="no"/>
-<layer number="4" name="Route4" color="1" fill="4" visible="no" active="no"/>
-<layer number="5" name="Route5" color="4" fill="4" visible="no" active="no"/>
-<layer number="6" name="Route6" color="1" fill="8" visible="no" active="no"/>
-<layer number="7" name="Route7" color="4" fill="8" visible="no" active="no"/>
-<layer number="8" name="Route8" color="1" fill="2" visible="no" active="no"/>
-<layer number="9" name="Route9" color="4" fill="2" visible="no" active="no"/>
-<layer number="10" name="Route10" color="1" fill="7" visible="no" active="no"/>
-<layer number="11" name="Route11" color="4" fill="7" visible="no" active="no"/>
-<layer number="12" name="Route12" color="1" fill="5" visible="no" active="no"/>
-<layer number="13" name="Route13" color="4" fill="5" visible="no" active="no"/>
-<layer number="14" name="Route14" color="1" fill="6" visible="no" active="no"/>
-<layer number="15" name="Route15" color="4" fill="6" visible="no" active="no"/>
-<layer number="16" name="Bottom" color="1" fill="1" visible="no" active="no"/>
-<layer number="17" name="Pads" color="2" fill="1" visible="no" active="no"/>
-<layer number="18" name="Vias" color="2" fill="1" visible="no" active="no"/>
-<layer number="19" name="Unrouted" color="6" fill="1" visible="no" active="no"/>
-<layer number="20" name="Dimension" color="15" fill="1" visible="no" active="no"/>
-<layer number="21" name="tPlace" color="7" fill="1" visible="no" active="no"/>
-<layer number="22" name="bPlace" color="7" fill="1" visible="no" active="no"/>
-<layer number="23" name="tOrigins" color="15" fill="1" visible="no" active="no"/>
-<layer number="24" name="bOrigins" color="15" fill="1" visible="no" active="no"/>
-<layer number="25" name="tNames" color="7" fill="1" visible="no" active="no"/>
-<layer number="26" name="bNames" color="7" fill="1" visible="no" active="no"/>
-<layer number="27" name="tValues" color="7" fill="1" visible="no" active="no"/>
-<layer number="28" name="bValues" color="7" fill="1" visible="no" active="no"/>
+<layer number="1" name="Top" color="4" fill="1" visible="yes" active="no"/>
+<layer number="2" name="Route2" color="1" fill="3" visible="yes" active="no"/>
+<layer number="3" name="Route3" color="4" fill="3" visible="yes" active="no"/>
+<layer number="4" name="Route4" color="1" fill="4" visible="yes" active="no"/>
+<layer number="5" name="Route5" color="4" fill="4" visible="yes" active="no"/>
+<layer number="6" name="Route6" color="1" fill="8" visible="yes" active="no"/>
+<layer number="7" name="Route7" color="4" fill="8" visible="yes" active="no"/>
+<layer number="8" name="Route8" color="1" fill="2" visible="yes" active="no"/>
+<layer number="9" name="Route9" color="4" fill="2" visible="yes" active="no"/>
+<layer number="10" name="Route10" color="1" fill="7" visible="yes" active="no"/>
+<layer number="11" name="Route11" color="4" fill="7" visible="yes" active="no"/>
+<layer number="12" name="Route12" color="1" fill="5" visible="yes" active="no"/>
+<layer number="13" name="Route13" color="4" fill="5" visible="yes" active="no"/>
+<layer number="14" name="Route14" color="1" fill="6" visible="yes" active="no"/>
+<layer number="15" name="Route15" color="4" fill="6" visible="yes" active="no"/>
+<layer number="16" name="Bottom" color="1" fill="1" visible="yes" active="no"/>
+<layer number="17" name="Pads" color="2" fill="1" visible="yes" active="no"/>
+<layer number="18" name="Vias" color="2" fill="1" visible="yes" active="no"/>
+<layer number="19" name="Unrouted" color="6" fill="1" visible="yes" active="no"/>
+<layer number="20" name="Dimension" color="15" fill="1" visible="yes" active="no"/>
+<layer number="21" name="tPlace" color="7" fill="1" visible="yes" active="no"/>
+<layer number="22" name="bPlace" color="7" fill="1" visible="yes" active="no"/>
+<layer number="23" name="tOrigins" color="15" fill="1" visible="yes" active="no"/>
+<layer number="24" name="bOrigins" color="15" fill="1" visible="yes" active="no"/>
+<layer number="25" name="tNames" color="7" fill="1" visible="yes" active="no"/>
+<layer number="26" name="bNames" color="7" fill="1" visible="yes" active="no"/>
+<layer number="27" name="tValues" color="7" fill="1" visible="yes" active="no"/>
+<layer number="28" name="bValues" color="7" fill="1" visible="yes" active="no"/>
 <layer number="29" name="tStop" color="7" fill="3" visible="no" active="no"/>
 <layer number="30" name="bStop" color="7" fill="6" visible="no" active="no"/>
@@
 <layer number="35" name="tGlue" color="7" fill="4" visible="no" active="no"/>
 <layer number="36" name="bGlue" color="7" fill="5" visible="no" active="no"/>
-<layer number="37" name="tTest" color="7" fill="1" visible="no" active="no"/>
-<layer number="38" name="bTest" color="7" fill="1" visible="no" active="no"/>
+<layer number="37" name="tTest" color="7" fill="1" visible="yes" active="no"/>
+<layer number="38" name="bTest" color="7" fill="1" visible="yes" active="no"/>
 <layer number="39" name="tKeepout" color="4" fill="11" visible="no" active="no"/>
 <layer number="40" name="bKeepout" color="1" fill="11" visible="no" active="no"/>
@@
 <layer number="44" name="Drills" color="7" fill="1" visible="no" active="no"/>
 <layer number="45" name="Holes" color="7" fill="1" visible="no" active="no"/>
-<layer number="46" name="Milling" color="3" fill="1" visible="no" active="no"/>
-<layer number="47" name="Measures" color="7" fill="1" visible="no" active="no"/>
-<layer number="48" name="Document" color="7" fill="1" visible="no" active="no"/>
-<layer number="49" name="Reference" color="7" fill="1" visible="no" active="no"/>
-<layer number="50" name="dxf" color="7" fill="1" visible="no" active="no"/>
-<layer number="51" name="tDocu" color="7" fill="1" visible="no" active="no"/>
-<layer number="52" name="bDocu" color="7" fill="1" visible="no" active="no"/>
-<layer number="53" name="tGND_GNDA" color="7" fill="1" visible="no" active="no"/>
-<layer number="54" name="bGND_GNDA" color="7" fill="1" visible="no" active="no"/>
-<layer number="56" name="wert" color="7" fill="1" visible="no" active="no"/>
-<layer number="57" name="tCAD" color="7" fill="1" visible="no" active="no"/>
-<layer number="59" name="tCarbon" color="7" fill="1" visible="no" active="no"/>
-<layer number="60" name="bCarbon" color="7" fill="1" visible="no" active="no"/>
+<layer number="46" name="Milling" color="3" fill="1" visible="yes" active="no"/>
+<layer number="47" name="Measures" color="7" fill="1" visible="yes" active="no"/>
+<layer number="48" name="Document" color="7" fill="1" visible="yes" active="no"/>
+<layer number="49" name="Reference" color="7" fill="1" visible="yes" active="no"/>
+<layer number="50" name="dxf" color="7" fill="1" visible="yes" active="no"/>
+<layer number="51" name="tDocu" color="7" fill="1" visible="yes" active="no"/>
+<layer number="52" name="bDocu" color="7" fill="1" visible="yes" active="no"/>
+<layer number="53" name="tGND_GNDA" color="7" fill="1" visible="yes" active="no"/>
+<layer number="54" name="bGND_GNDA" color="7" fill="1" visible="yes" active="no"/>
+<layer number="56" name="wert" color="7" fill="1" visible="yes" active="no"/>
+<layer number="57" name="tCAD" color="7" fill="1" visible="yes" active="no"/>
+<layer number="59" name="tCarbon" color="7" fill="1" visible="yes" active="no"/>
+<layer number="60" name="bCarbon" color="7" fill="1" visible="yes" active="no"/>
 <layer number="90" name="Modules" color="5" fill="1" visible="yes" active="yes"/>
 <layer number="91" name="Nets" color="2" fill="1" visible="yes" active="yes"/>
@@
 <part name="JP2" library="holla" deviceset="JUMPER-PAD-2-NO" device="" value="DNP"/>
 <part name="GND10" library="holla" deviceset="GND" device=""/>
-<part name="R73" library="holla" deviceset="R" device="-0603" value="3.9k"/>
-<part name="R74" library="holla" deviceset="R" device="-0603" value="3.9k"/>
+<part name="R73" library="holla" deviceset="R" device="-0603" value="1k"/>
+<part name="R74" library="holla" deviceset="R" device="-0603" value="1k"/>
 <part name="R17" library="holla" deviceset="R" device="-0603" value="1k"/>
 <part name="D3" library="holla" deviceset="LED" device="-0603" value="GRN"/>
@@
 <part name="GND2" library="holla" deviceset="GND" device=""/>
 <part name="J11" library="holla" deviceset="CONN-04" device="-0.1"/>
-<part name="R39" library="holla" deviceset="R" device="-0603" value="120"/>
-<part name="R40" library="holla" deviceset="R" device="-0603" value="120"/>
+<part name="R39" library="holla" deviceset="R" device="-0603" value="1k"/>
+<part name="R40" library="holla" deviceset="R" device="-0603" value="1k"/>
 <part name="R78" library="holla" deviceset="R" device="-0603" value="120"/>
 <part name="C15" library="holla" deviceset="C" device="-0603" value=".1u"/>

Commit message: initial add for blink
Parts:
- added U22: DUALOPAMP, holla:AMP-OPAMP-DUAL-SO08
- B1: value CONN-COINBATTERYHOLDER-20MM -> CR2032
- D35, D36: device holla:DIODE-0805 -> holla:DIODE-0603
- Q1, Q2, Q3, Q4: value IRFZ44 -> FET-NCH
- Q10, Q21, Q22, Q23, Q24, Q25, Q26, Q27, Q28, Q29, Q30, Q5, Q6, Q7, Q8, Q9: value FDD4141 -> FET-PCH
- Q11, Q12, Q13, Q14, Q15, Q16, Q17, Q18, Q19, Q20, Q31, Q32, Q33, Q34, Q35, Q36, Q37, Q38, Q39, Q40, Q42, Q43, Q44, Q45, Q46, Q47: value 2N7002 -> FET-NCH
- Q41: value FDD4141 -> FET-PCH; device brightleaf:FDD4141TO252 -> brightleaf:FET-PCHTO252
- S1, S2: value (none) -> UI
- U12, U13, U14, U15: value OPTO-LTV817 -> OPTO
Other:
- note added: "Description The Tex Hat is a multi-purpose expansion board. This page is overall block diagram. Each page contains brief descriptions outlining individual functionality. The board does not require full component population to function. System designers can pick and choose what capabilities required. Also, see "use cases.ods" for additional functionality descriptions. TODO Make all diodes the same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"
- note added: "I2C Address Table 0x20 010 0000 I/O MCP23107 0x40 100 0000 VBATT Current Sense INA219 0x48 100 1000 ADC ADS1015 0x4C 100 1100 TEMP LM75 0x60 110 0000 LED PCA9685 0x6F 110 1111 RTC MCP7940 0x78 111 1000 Display SSD1306 Banggood"
- note removed: "Description The Tex Hat is a multi-purpose expansion board. This page is overall block diagram. Each page contains brief descriptions outlining individual functionality. The board does not require full component population to function. System designers can pick and choose what capabilities required. Also, see "use cases.ods" for additional functionality descriptions."
- note removed: "I2C Address Table 010 0000 I/O MCP23107 100 0000 VBATT Current Sense INA219 100 1000 ADC ADS1015 100 1100 TEMP LM75 110 0000 LED PCA9685 110 1111 RTC MCP7940 111 1000 Display SSD1306 Banggood"

Commit message: added todo items
Parts:
- F1: value 20A -> 10A
- R33, R34: value 1 -> 0.1
- R51: value 10 -> 0.1
Other:
- note added: "I2C Address Table 0x20 010 0000 I/O MCP23107 0x40 100 0000 VBATT Current Sense INA219 0x48 100 1000 ADC ADS1015 0x4C 100 1100 TEMP LM75 0x60 110 0000 LED PCA9685 0x6F 110 1111 RTC MCP7940 0x78 111 1000 Display SSD1306 Banggood pi@raspberrypi: i2cdetect -y 1 0 1 2 3 4 5 6 7 8 9 a b c d e f 00: -- -- -- -- -- -- -- -- -- -- -- -- -- 10: -- -- -- -- -- -- -- -- -- -- -- -- -- -- -- -- 20: 20 -- -- -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"
- note removed: "I2C Address Table 0x20 010 0000 I/O MCP23107 0x40 100 0000 VBATT Current Sense INA219 0x48 100 1000 ADC ADS1015 0x4C 100 1100 TEMP LM75 0x60 110 0000 LED PCA9685 0x6F 110 1111 RTC MCP7940 0x78 111 1000 Display SSD1306 Banggood"
Changed lines of the file:
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@@
 <part name="GND14" library="holla" deviceset="GND" device=""/>
 <part name="GND15" library="holla" deviceset="GND" device=""/>
-<part name="F1" library="holla" deviceset="FUSE-HOLDER" device="-3557-2" value="20A"/>
+<part name="F1" library="holla" deviceset="FUSE-HOLDER" device="-3557-2" value="10A"/>
 <part name="GND1" library="holla" deviceset="GND" device=""/>
 <part name="C16" library="holla" deviceset="C" device="-0603" value=".1u"/>
@@
 <part name="Q1" library="holla" deviceset="FET-NCHANNEL" device="-TO252" value="FET-NCH"/>
 <part name="GND45" library="holla" deviceset="GND" device=""/>
-<part name="R33" library="holla" deviceset="R" device="-1210" value="1"/>
+<part name="R33" library="holla" deviceset="R" device="-1210" value="0.1"/>
 <part name="Q24" library="holla" deviceset="FET-PCHANNEL" device="-TO252" value="FET-PCH"/>
 <part name="R35" library="holla" deviceset="R" device="-0603" value="47k"/>
@@
 <part name="Q3" library="holla" deviceset="FET-NCHANNEL" device="-TO252" value="FET-NCH"/>
 <part name="GND43" library="holla" deviceset="GND" device=""/>
-<part name="R34" library="holla" deviceset="R" device="-1210" value="1"/>
+<part name="R34" library="holla" deviceset="R" device="-1210" value="0.1"/>
 <part name="R18" library="holla" deviceset="R" device="-0603" value="1k"/>
 <part name="D18" library="holla" deviceset="LED" device="-0603" value="RED"/>
@@
 <part name="D1" library="holla" deviceset="LED" device="-0603" value="GRN"/>
 <part name="GND40" library="holla" deviceset="GND" device=""/>
-<part name="R51" library="holla" deviceset="R" device="-1210" value="10"/>
+<part name="R51" library="holla" deviceset="R" device="-1210" value="0.1"/>
 <part name="J20" library="holla" deviceset="CONN-02" device="-6.35MM"/>
 <part name="J4" library="holla" deviceset="CONN-04" device="-PLUGIN-SCREW"/>
@@
 <wire x1="172.72" y1="141.605" x2="242.57" y2="141.605" width="0.1524" layer="94"/>
 <wire x1="242.57" y1="141.605" x2="242.57" y2="132.715" width="0.1524" layer="94"/>
-<text x="58.42" y="195.58" size="1.778" layer="97" align="top-left">Description
+<text x="7.62" y="208.28" size="1.778" layer="97" align="top-left">Description
 The Tex Hat is a multi-purpose expansion board. This page is
 overall block diagram. Each page contains brief descriptions
@@
 Also, see "use cases.ods" for additional functionality descriptions.
 TODO
-Make all diodes the same package</text>
+Make all diodes the same package
+The board's RPI mounting holes need to be 3.5mm dia
+Add battery polarity in SS
+Add connector labels
+Add pull-down to turn relays off until the 23017 turns pins as output</text>
 <text x="136.906" y="132.08" size="1.016" layer="94" rot="R180" align="center">ISENSE</text>
 <wire x1="140.97" y1="130.81" x2="135.89" y2="130.81" width="0.1524" layer="94"/>
@@
  0x6F 110 1111 RTC MCP7940
  0x78 111 1000 Display SSD1306 Banggood
+pi@raspberrypi: i2cdetect -y 1
+     0  1  2  3  4  5  6  7  8  9  a  b  c  d  e  f
+00:          -- -- -- -- -- -- -- -- -- -- -- -- --
+10: -- -- -- -- -- -- -- -- -- -- -- -- -- -- -- --
+20: 20 -- -- -- -- -- -- -- -- -- -- -- -- -- -- --
+30: -- -- -- -- -- -- -- -- -- -- -- -- 3c -- -- --
+40: 40 -- -- -- -- -- -- -- 48 -- -- -- 4c -- -- --
+50: -- -- -- -- -- -- -- -- -- -- -- -- -- -- -- --
+60: 60 -- -- -- -- -- -- -- -- -- -- -- -- -- -- 6f
+70: 70 -- -- -- -- -- -- --
 </text>
 <text x="114.554" y="100.33" size="1.016" layer="94" rot="R180" align="center">RELAY</text>
