File: board/tex.sch (EAGLE design)
At the start: 271 parts, among them Q1 FET-NCH, Q10 FET-PCH, Q11 FET-NCH, Q12 FET-NCH, Q13 FET-NCH, Q14 FET-NCH, Q15 FET-NCH, Q16 FET-NCH, Q17 FET-NCH, Q18 FET-NCH, Q19 FET-NCH, Q2 FET-NCH, Q20 FET-NCH, Q21 FET-PCH, Q22 FET-PCH, Q23 FET-PCH, Q24 FET-PCH, Q25 FET-PCH, Q26 FET-PCH, Q27 FET-PCH, Q28 FET-PCH, Q29 FET-PCH, Q3 FET-NCH, Q30 FET-PCH, Q31 FET-NCH, Q32 FET-NCH, Q33 FET-NCH, Q34 FET-NCH, Q35 FET-NCH, Q36 FET-NCH, Q37 FET-NCH, Q38 FET-NCH, Q39 FET-NCH, Q4 FET-NCH, Q40 FET-NCH, Q41 FET-PCH, Q42 FET-NCH, Q43 FET-NCH, Q44 FET-NCH, Q45 FET-NCH, Q46 FET-NCH, Q47 FET-NCH, Q5 FET-PCH, Q6 FET-PCH, Q7 FET-PCH, Q8 FET-PCH, Q9 FET-PCH, U10 ADS1x15, U11 DUALOPAMP, U12 OPTO, U13 OPTO, U14 OPTO, U15 OPTO, U16 MCP23017, U17 24LC32A, U18 IO-HC4051, U19 MCP7940N, U22 DUALOPAMP, U3 MAX13433E, U4 AZ23C5V1, U5 PCA9685, U6 DUALOPAMP, U7 INA219, U8 LM75, Y1 32.768KHz

Commit message: added more notes
Other:
- note added: "I2C Address Table 0x20 010 0000 I/O MCP23107 0x3C 011 1100 128x64 OLED Display SSD1306 0x40 100 0000 VBATT Current Sense INA219 0x48 100 1000 ADC ADS1015 0x4C 100 1100 TEMP LM75 0x60 110 0000 LED PCA9685 0x6F 110 1111 RTC MCP7940 0x70 111 0000 unknown, might be RTC BB RAM pi@raspberrypi: i2cdetect -y 1 0 1 2 3 4 5 6 7 8 9 a b c d e f 00: -- -- -- -- -- -- -- -- -- -- -- -- -- 10: -- -- -- -- -- -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"
- note added: "addr 011 1100"
- note removed: "I2C Address Table 0x20 010 0000 I/O MCP23107 0x40 100 0000 VBATT Current Sense INA219 0x48 100 1000 ADC ADS1015 0x4C 100 1100 TEMP LM75 0x60 110 0000 LED PCA9685 0x6F 110 1111 RTC MCP7940 0x78 111 1000 Display SSD1306 Banggood pi@raspberrypi: i2cdetect -y 1 0 1 2 3 4 5 6 7 8 9 a b c d e f 00: -- -- -- -- -- -- -- -- -- -- -- -- -- 10: -- -- -- -- -- -- -- -- -- -- -- -- -- -- -- -- 20: 20 -- -- -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"
- note removed: "addr 111 1000"
Changed lines of the file:
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@@
 <wire x1="160.02" y1="133.35" x2="160.02" y2="135.89" width="0.1524" layer="94"/>
 <circle x="143.51" y="132.08" radius="0.127" width="0.4064" layer="94"/>
-<circle x="142.24" y="138.43" radius="0.127" width="0.4064" layer="94"/>
 <circle x="205.74" y="132.08" radius="0.127" width="0.4064" layer="94"/>
 <circle x="208.28" y="132.08" radius="0.127" width="0.4064" layer="94"/>
@@
 <wire x1="165.1" y1="157.48" x2="162.56" y2="157.48" width="0.1524" layer="94"/>
 <wire x1="162.56" y1="157.48" x2="162.56" y2="160.02" width="0.1524" layer="94"/>
-<wire x1="161.29" y1="144.78" x2="142.24" y2="144.78" width="0.1524" layer="94" style="shortdash"/>
-<wire x1="142.24" y1="144.78" x2="142.24" y2="138.43" width="0.1524" layer="94"/>
 <wire x1="151.13" y1="135.89" x2="151.13" y2="137.16" width="0.1524" layer="94"/>
 <wire x1="151.13" y1="137.16" x2="143.51" y2="137.16" width="0.1524" layer="94"/>
@@
 <text x="22.86" y="83.82" size="2.54" layer="97" align="top-left">I2C Address Table
  0x20 010 0000 I/O MCP23107
+ 0x3C 011 1100 128x64 OLED Display SSD1306
  0x40 100 0000 VBATT Current Sense INA219
  0x48 100 1000 ADC ADS1015
@@
  0x60 110 0000 LED PCA9685
  0x6F 110 1111 RTC MCP7940
- 0x78 111 1000 Display SSD1306 Banggood
+ 0x70 111 0000 unknown, might be RTC BB RAM
 pi@raspberrypi: i2cdetect -y 1
      0  1  2  3  4  5  6  7  8  9  a  b  c  d  e  f
@@
 <wire x1="166.37" y1="139.7" x2="166.37" y2="157.48" width="0.1524" layer="94"/>
 <wire x1="165.1" y1="139.7" x2="165.1" y2="157.48" width="0.1524" layer="94"/>
-<wire x1="161.29" y1="139.7" x2="161.29" y2="144.78" width="0.1524" layer="94"/>
 <wire x1="161.29" y1="161.29" x2="170.18" y2="161.29" width="0.1524" layer="94"/>
 <wire x1="170.18" y1="161.29" x2="170.18" y2="160.02" width="0.1524" layer="94"/>
@@
 <text x="33.02" y="55.88" size="1.778" layer="97">addr 100 1100</text>
 <text x="137.16" y="7.62" size="1.778" layer="97">addr 110 1111</text>
-<text x="60.96" y="22.86" size="1.778" layer="97">addr 111 1000</text>
+<text x="60.96" y="22.86" size="1.778" layer="97">addr 011 1100</text>
 <text x="11.684" y="136.144" size="1.27" layer="97" align="top-left">Description
 U3 is a full-duplex differential line driver

Commit message: more notes
Parts:
- C13, C14: value 12p -> 6p
Other:
- note added: "12p not recommended for 7940"
Changed lines of the file:
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@@
 <part name="R79" library="holla" deviceset="R" device="-0603" value="120"/>
 <part name="GND4" library="holla" deviceset="GND" device=""/>
-<part name="C13" library="holla" deviceset="C" device="-0603" value="12p"/>
-<part name="C14" library="holla" deviceset="C" device="-0603" value="12p"/>
+<part name="C13" library="holla" deviceset="C" device="-0603" value="6p"/>
+<part name="C14" library="holla" deviceset="C" device="-0603" value="6p"/>
 <part name="GND2" library="holla" deviceset="GND" device=""/>
 <part name="J11" library="holla" deviceset="CONN-04" device="-0.1"/>
@@
 during linux startup hardware discovery
 phase. It is optional.</text>
+<text x="101.6" y="10.16" size="1.778" layer="97">12p not recommended
+for 7940</text>
 </plain>
 <instances>
